File: Mirobot.kicad_pcb (KiCad board)
At the start: 2 copper layers, 110 x 31.5 mm, 49 parts, among them M1 ESP8266-ESP-12, P1 USB_OTG, P2 RIGHT_STEPPER, P3 LEFT_STEPPER, P4 CONN_01X06, Q1 S8050, Q2 S8050, Q3 S8050, SW1 LEFT_BUMP, SW2 RIGHT_BUMP, SW3 POWER_SWITCH, U1 phototransistor, U2 phototransistor, U3 PCF8591, U4 74HC595, U5 ULN2803A, U6 CP2104, U8 LD1117S33CTR

Commit message: v3.1 of the PCB
Parts:
- F1: value FUSE -> 1A
- P2: value RIGHT_STEPPER -> STEPPER
- P3: value LEFT_STEPPER -> STEPPER
- P4: moved to B.Cu
- R10: value 10K -> 10k
- SW1: value LEFT_BUMP -> COLLISION
- SW2: value RIGHT_BUMP -> COLLISION
- turned P4 to 270 degrees
Connections:
- M1 pad 10: SERVO -> LED
- M1 pad 13: LED -> SERVO
- R3 pad 2: SERVO -> LED
Routing:
- net LED: track 11.4 -> 39.7 mm, vias 2 -> 4
- net SERVO: track 42.0 -> 49.1 mm
- net GND: track 105.3 -> 108.1 mm
- net Net-(R6-Pad1): track 32.8 -> 33.3 mm

Commit message: v3.2 of the PCB
Parts:
- removed Q3: S8050, Custom:SOT-23
- removed R13: 10k, Resistors_SMD:R_0603
- removed R9: 160R, Resistors_SMD:R_0603
- added C2: 0.1uF, Capacitors_SMD:C_0603, B.Cu at (128.7, 138.9)
- added P5: CONN_01X04, Pin_Headers:Pin_Header_Straight_1x04, F.Cu at (165.2, 149.5)
- added R14: 27R, Resistors_SMD:R_0603, B.Cu at (120.1, 133.5)
- added R15: 27R, Resistors_SMD:R_0603, B.Cu at (126.0, 133.5)
- added R16: 1.5k, Resistors_SMD:R_0603, B.Cu at (123.1, 133.5)
- C4: value 4.7uF -> 0.1uF
- P4: footprint Pin_Headers:Pin_Header_Straight_1x06 -> Custom:6-PIN-EDGE-CONN
- U6: value CP2104 -> PL2303HX; footprint Custom:QFN-24-1EP_4x4mm_Pitch0.5mm-easySolder -> Housings_SSOP:SSOP-28_5.3x10.2mm_Pitch0.65mm
- moved FID3 93.3 mm to (209.9, 144.8)
- moved C4 9.43 mm to (117.5, 143.6), turned to 90 degrees
- moved P4 8.25 mm to (115.2, 139.0), turned to 90 degrees
- moved R10 7.96 mm to (128.7, 141.9), turned to 270 degrees
- moved C3 7.65 mm to (117.5, 140.1), turned to 90 degrees
- moved C1 1.75 mm to (204.8, 140.7)
- moved U6 1.32 mm to (123.0, 140.0), turned to 180 degrees
- moved Q1 0.89 mm to (131.3, 135.8)
- moved Q2 0.89 mm to (131.3, 141.9)
- moved R11 0.89 mm to (132.3, 138.8)
- moved R12 0.89 mm to (130.4, 138.8)
Connections:
- C3 pad 1: +3V3 -> +5V
- C4 pad 1: +3V3 -> GND
- C4 pad 2: GND -> Net-(C4-Pad2)
- D2 pad 1: Net-(D1-Pad1) -> LED_EN
- D2 pad 2: Net-(D2-Pad2) -> Net-(D1-Pad1)
- P4 pad 2: SCL -> Net-(P4-Pad2)
- P4 pad 3: +3V3 -> +5V
- P4 pad 6: RESET -> Net-(P4-Pad6)
- Q1 pad 1: Net-(Q1-Pad1) -> Net-(P4-Pad6)
- Q1 pad 3: SCL -> SDA
- Q2 pad 1: Net-(Q2-Pad1) -> Net-(P4-Pad2)
- R11 pad 1: Net-(Q2-Pad1) -> Net-(P4-Pad2)
- R12 pad 1: Net-(Q1-Pad1) -> Net-(P4-Pad6)
- U6 pad 1: Net-(U6-Pad1) -> RXD
- U6 pad 10: Net-(U6-Pad10) -> Net-(R10-Pad2)
- U6 pad 16: GND -> Net-(R14-Pad2)
- U6 pad 17: Net-(U6-Pad17) -> Net-(C4-Pad2)
- U6 pad 18: Net-(U6-Pad18) -> GND
- U6 pad 19: Net-(Q2-Pad1) -> Net-(C4-Pad2)
- U6 pad 2: GND -> Net-(P4-Pad6)
- U6 pad 20: TXD -> +5V
- U6 pad 21: RXD -> Net-(U6-Pad21)
- U6 pad 23: Net-(Q1-Pad1) -> Net-(U6-Pad23)
- U6 pad 3: Net-(P1-Pad3) -> Net-(P4-Pad2)
- U6 pad 4: Net-(P1-Pad2) -> +3V3
- U6 pad 5: +3V3 -> TXD
- U6 pad 6: +3V3 -> Net-(U6-Pad6)
- U6 pad 7: +3V3 -> GND
- U6 pad 9: Net-(R10-Pad2) -> Net-(U6-Pad9)
Routing:
- net +5V: track 41.1 -> 89.1 mm, vias 1 -> 2
- net SCL: track 66.3 -> 26.4 mm, vias 0 -> 1
- net SDA: track 16.5 -> 50.6 mm, vias 0 -> 1
- net Net-(P4-Pad2): track 0.00 -> 24.7 mm, vias 0 -> 2
- net Net-(P1-Pad3): track 52.4 -> 30.4 mm
- net Net-(C4-Pad2): track 0.00 -> 20.1 mm
- net Net-(P4-Pad6): track 0.00 -> 19.7 mm, vias 0 -> 2
- net Net-(R15-Pad2): track 0.00 -> 16.4 mm
- net Net-(D2-Pad2): track 14.7 -> 0.00 mm
- net Net-(Q1-Pad1): track 13.6 -> 0.00 mm
- net Net-(R14-Pad2): track 0.00 -> 13.2 mm
- net Net-(P1-Pad2): track 47.4 -> 34.2 mm
- net Net-(Q2-Pad1): track 9.83 -> 0.00 mm, vias 2 -> 0
- net TXD: track 66.7 -> 58.3 mm
- net RXD: track 60.8 -> 52.6 mm, vias 0 -> 2
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Other:
- board text added: "3.3V"
- board text added: "GND"
- board text added: "PCB v3.2"
- board text added: "SCL"
- board text added: "SDA"
- board text added: "v3"
- board text removed: "v3.1"

Commit message: v3.3 of the PCB
Parts:
- removed C4: 0.1uF, Capacitors_SMD:C_0603
- removed R10: 10k, Resistors_SMD:R_0603
- removed R14, R15: 27R, Resistors_SMD:R_0603
- removed R16: 1.5k, Resistors_SMD:R_0603
- added X1: 12MHz, Crystals:crystal_FA238-TSX3225, B.Cu at (116.6, 138.2)
- BATT1: footprint Pin_Headers:Pin_Header_Straight_1x02 -> Custom:JST_XH-1x02
- C2, C3: value 0.1uF -> 22pF
- M1: footprint Custom:ESP-07 -> Custom:ESP-12
- P5: moved to B.Cu
- U6: value PL2303HX -> CH340G; footprint Housings_SSOP:SSOP-28_5.3x10.2mm_Pitch0.65mm -> SMD_Packages:SO-16-N
- moved C2 12.6 mm to (116.6, 135.0), turned to 180 degrees
- moved P4 10.4 mm to (123.3, 145.6), turned to 180 degrees
- moved Q1 6.37 mm to (131.9, 142.1), turned to 0 degrees
- moved Q2 5.87 mm to (131.9, 136.0), turned to 180 degrees
- moved FID1 5.04 mm to (123.0, 122.9)
- moved FID2 4.99 mm to (214.9, 123.0)
- moved FID3 4.98 mm to (214.9, 144.8)
- moved P1 4.19 mm to (145.9, 125.4)
- moved SW3 2.84 mm to (188.6, 122.4)
- moved L1 2.56 mm to (155.3, 123.1), turned to 180 degrees
- moved R12 2.49 mm to (132.8, 139.1), turned to 90 degrees
- moved C1 2.31 mm to (206.9, 139.8)
- moved D2 2.13 mm to (184.9, 150.0), turned to 270 degrees
- moved D1 2.10 mm to (152.9, 150.0), turned to 270 degrees
- moved U6 2.07 mm to (123.7, 138.0)
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Connections:
- C2 pad 1: +3V3 -> Net-(C2-Pad1)
- C3 pad 1: +5V -> Net-(C3-Pad1)
- U6 pad 1: RXD -> GND
- U6 pad 13: Net-(U6-Pad13) -> Net-(P4-Pad6)
- U6 pad 14: Net-(U6-Pad14) -> Net-(P4-Pad2)
- U6 pad 16: Net-(R14-Pad2) -> +3V3
- U6 pad 2: Net-(P4-Pad6) -> RXD
- U6 pad 3: Net-(P4-Pad2) -> TXD
- U6 pad 5: TXD -> Net-(P1-Pad3)
- U6 pad 6: Net-(U6-Pad6) -> Net-(P1-Pad2)
- U6 pad 7: GND -> Net-(C2-Pad1)
- U6 pad 8: Net-(U6-Pad8) -> Net-(C3-Pad1)
Routing:
- net GND: track 113.0 -> 73.0 mm, vias 24 -> 22
- net Net-(C4-Pad2): track 20.1 -> 0.00 mm
- net Net-(U6-Pad15): track 16.4 -> 0.00 mm
- net Net-(R14-Pad2): track 13.2 -> 0.00 mm
- net Net-(C3-Pad1): track 0.00 -> 8.43 mm
- net Net-(C2-Pad1): track 0.00 -> 7.99 mm
- net Net-(P4-Pad6): track 19.7 -> 27.6 mm, vias 2 -> 0
- net Net-(P4-Pad2): track 24.7 -> 16.8 mm
- net +3V3: track 208.9 -> 201.8 mm, vias 4 -> 5
- net Net-(D1-Pad1): track 34.8 -> 29.5 mm
- net +5V: track 89.1 -> 93.6 mm
- net LED: track 42.7 -> 46.8 mm
- net Net-(P1-Pad3): track 30.4 -> 33.8 mm
- net Net-(D1-Pad2): track 15.7 -> 12.5 mm
- net LED_EN: track 29.9 -> 27.1 mm
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Other:
- outline, holes or cut-outs redrawn
- board text added: "74HC595"
- board text added: "CH340G"
- board text added: "PCB v3.3"
- board text added: "PCF8591"
- board text added: "ULN2803"
- board text added: "V"
- board text removed: "PCB v3.2"

Commit message: v3.4 of the PCB
Parts:
- moved P1 29.4 mm to (121.5, 142.0), turned to 180 degrees
- moved P4 25.5 mm to (132.3, 121.8)
- moved SW3 2.43 mm to (186.2, 122.7)
- moved C2 2.29 mm to (116.6, 132.8)
- moved C3 2.29 mm to (116.6, 138.8)
- moved Q1 2.29 mm to (131.8, 139.8)
- moved Q2 2.29 mm to (131.8, 133.7)
- moved R11 2.29 mm to (130.9, 136.8)
- moved R12 2.29 mm to (132.8, 136.8)
- moved X1 2.29 mm to (116.5, 135.9)
- moved U6 2.29 mm to (123.6, 135.8)
- moved L1 1.21 mm to (156.5, 123.1)
- moved M1 0.25 mm to (170.2, 134.9)
Routing:
- net Net-(P1-Pad2): track 36.5 -> 2.74 mm
- net Net-(P1-Pad3): track 33.8 -> 5.73 mm
- net RXD: track 50.9 -> 70.4 mm, vias 0 -> 2
- net Net-(P4-Pad2): track 16.8 -> 34.5 mm
- net +5V: track 93.6 -> 105.2 mm
- net TXD: track 58.7 -> 68.3 mm
- net Net-(P4-Pad6): track 27.6 -> 24.3 mm
- net Net-(BATT1-Pad2): track 22.6 -> 25.3 mm
- net Net-(F1-Pad1): track 30.6 -> 33.2 mm, vias 0 -> 1
- net LED: track 46.8 -> 45.0 mm
- net RESET: track 61.7 -> 63.2 mm
- net SDA: track 52.2 -> 51.2 mm
- net +3V3: track 201.8 -> 202.4 mm
- net GND: track 73.0 -> 73.4 mm, vias 22 -> 20
Other:
- outline, holes or cut-outs redrawn
- board text added: "PCB v3.4"
- board text added: "•"
- board text removed: "PCB v3.3"
- board text removed: "V"

Commit message: v3.5 of the PCB
Parts:
- added W1: TEST_1P, Measurement_Points:Measurement_Point_Round-SMD-Pad_Small, F.Cu at (157.9, 127.6)
- added W2: TEST_1P, Measurement_Points:Measurement_Point_Round-SMD-Pad_Small, F.Cu at (128.7, 135.6)
- added W3: TEST_1P, Measurement_Points:Measurement_Point_Round-SMD-Pad_Small, F.Cu at (126.2, 135.6)
- added W4: TEST_1P, Measurement_Points:Measurement_Point_Round-SMD-Pad_Small, F.Cu at (166.2, 146.1)
- added W5: TEST_1P, Measurement_Points:Measurement_Point_Round-SMD-Pad_Small, F.Cu at (123.6, 135.6)
- added W6: TEST_1P, Measurement_Points:Measurement_Point_Round-SMD-Pad_Small, F.Cu at (121.1, 135.6)
- added W7: TEST_1P, Measurement_Points:Measurement_Point_Round-SMD-Pad_Small, F.Cu at (118.6, 135.6)
- added W8: TEST_1P, Measurement_Points:Measurement_Point_Round-SMD-Pad_Small, F.Cu at (130.4, 141.8)
- ART1: footprint Custom:MIROBOT_LOGO -> Custom:MIME_MIROBOT_LOGO
- BATT1: footprint Custom:JST_XH-1x02 -> Connectors_JST:JST_PH_B3B-PH-K_03x2.00mm_Straight
- P4: value CONN_01X06 -> CONN_01X03; footprint Custom:6-PIN-EDGE-CONN -> Pin_Headers:Pin_Header_Straight_1x03
- moved F1 83.1 mm to (130.7, 140.2), turned to 90 degrees
- moved U8 76.0 mm to (142.9, 141.4), turned to 0 degrees
- moved BATT1 73.5 mm to (132.1, 130.3)
- moved C8 72.0 mm to (141.1, 135.2), turned to 180 degrees
- moved C1 71.5 mm to (135.4, 137.4), turned to 270 degrees
- moved PEN1 70.8 mm to (205.8, 130.5)
- moved SG1 68.2 mm to (208.4, 139.8)
- moved C6 68.0 mm to (144.9, 135.2), turned to 180 degrees
- moved SW3 59.9 mm to (130.4, 144.6), turned to 180 degrees
- moved Q1 26.2 mm to (157.3, 133.7)
- moved Q2 26.2 mm to (157.3, 127.6)
- moved R11 26.2 mm to (156.3, 130.6)
- moved R12 26.2 mm to (158.2, 130.6)
- moved ART1 21.4 mm to (146.6, 143.5)
- moved P4 12.3 mm to (144.6, 123.1), turned to 270 degrees
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Connections:
- BATT1 pad 2: Net-(BATT1-Pad2) -> +5V
- M1 pad 2: ADC -> (no net)
- P1 pad 4: Net-(P1-Pad4) -> (no net)
- P4 pad 1: GND -> Net-(L1-Pad2)
- P4 pad 2: Net-(P4-Pad2) -> GND
- P4 pad 3: +5V -> +3V3
- Q1 pad 1: Net-(P4-Pad6) -> Net-(Q1-Pad1)
- Q2 pad 1: Net-(P4-Pad2) -> Net-(Q2-Pad1)
- R11 pad 1: Net-(P4-Pad2) -> Net-(Q2-Pad1)
- R12 pad 1: Net-(P4-Pad6) -> Net-(Q1-Pad1)
- SW3 pad 1: Net-(BATT1-Pad2) -> +5V
- SW3 pad 3: +5V -> Net-(BATT1-Pad3)
- U3 pad 11: Net-(U3-Pad11) -> (no net)
- U3 pad 15: Net-(U3-Pad15) -> (no net)
- U4 pad 16: VCC -> (no net)
- U4 pad 9: Net-(U4-Pad9) -> (no net)
- U6 pad 10: Net-(U6-Pad10) -> (no net)
- U6 pad 11: Net-(U6-Pad11) -> (no net)
- U6 pad 12: Net-(U6-Pad12) -> (no net)
- U6 pad 13: Net-(P4-Pad6) -> Net-(Q1-Pad1)
- U6 pad 14: Net-(P4-Pad2) -> Net-(Q2-Pad1)
- U6 pad 15: Net-(U6-Pad15) -> (no net)
- U6 pad 9: Net-(U6-Pad9) -> (no net)
Routing:
- net +5V: track 105.2 -> 27.9 mm, vias 2 -> 0
- net Net-(Q1-Pad1): track 0.00 -> 42.1 mm
- net Net-(Q2-Pad1): track 0.00 -> 37.1 mm
- net Net-(P4-Pad2): track 34.5 -> 0.00 mm, vias 2 -> 0
- net RESET: track 63.2 -> 30.0 mm
- net Net-(F1-Pad1): track 33.2 -> 6.12 mm, vias 1 -> 0
- net SDA: track 51.2 -> 24.4 mm
- net RXD: track 70.4 -> 43.8 mm
- net Net-(BATT1-Pad2): track 25.3 -> 0.00 mm
- net Net-(P4-Pad6): track 24.3 -> 0.00 mm
- net TXD: track 68.3 -> 45.6 mm
- net BUZZER: track 33.7 -> 55.2 mm
- net +3V3: track 202.4 -> 223.8 mm, vias 5 -> 4
- net Net-(L1-Pad2): track 0.00 -> 16.7 mm, vias 0 -> 1
- net Net-(BATT1-Pad3): track 0.00 -> 15.8 mm
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Other:
- outline, holes or cut-outs redrawn
- board text added: "BATT ON"
- board text added: "DATA"
- board text added: "EXT LED"
- board text added: "GPIO0"
- board text added: "PCB v3.5"
- board text added: "RST"
- board text added: "RX"
- board text added: "TX"
- board text added: "USB+"
- board text added: "USB-"
- board text added: "VSS"
- board text added: "© 2017 Mime Industries http://mime.co.uk"
- board text removed: "-"
- board text removed: "B"
- board text removed: "BATT"
- board text removed: "PCB v3.4"
- board text removed: "POWER"
- board text removed: "http://mirobot.io © 2015 Ben Pirt"

Commit message: v3.6 of the PCB
Routing:
- net TXD: track 45.6 -> 46.5 mm
Other:
- board text added: "PCB v3.6"
- board text removed: "PCB v3.5"
Changed lines of the file:
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@@
   (general
     (links 137)
-    (no_connects 3)
+    (no_connects 0)
     (area 103.320999 116.0069 244.769467 158.789715)
     (thickness 1.6)
     (drawings 70)
-    (tracks 653)
+    (tracks 663)
     (zones 0)
     (modules 55)
@@
       (drillshape 0)
       (scaleselection 1)
-      (outputdirectory output/v3.5/))
+      (outputdirectory output/v3.6/))
   )
   (net 0 "")
@@
     (effects (font (size 1.5 1.5) (thickness 0.3)) (justify mirror))
   )
-  (gr_text "PCB v3.5\n" (at 151.892 134.239) (layer B.SilkS)
+  (gr_text "PCB v3.6\n" (at 151.892 134.239) (layer B.SilkS)
     (effects (font (size 1 1) (thickness 0.2)) (justify mirror))
   )
@@
   (segment (start 152.527 148.0185) (end 151.16 149.3855) (width 0.254) (layer B.Cu) (net 8))
   (segment (start 151.16 149.3855) (end 151.16 150) (width 0.254) (layer B.Cu) (net 8))
+  (segment (start 157.9 127.63) (end 157.9 126.912) (width 0.254) (layer F.Cu) (net 9))
+  (segment (start 157.9 126.912) (end 156.47 125.482) (width 0.254) (layer F.Cu) (net 9))
+  (segment (start 156.47 125.482) (end 156.47 125.45) (width 0.254) (layer F.Cu) (net 9))
   (segment (start 158.96066 127.63) (end 157.9 127.63) (width 0.254) (layer F.Cu) (net 9))
   (segment (start 173.5 127.63) (end 158.96066 127.63) (width 0.254) (layer F.Cu) (net 9))
   (segment (start 174.77 128.9) (end 173.5 127.63) (width 0.254) (layer F.Cu) (net 9))
-  (segment (start 157.9 127.63) (end 156.47 126.2) (width 0.254) (layer F.Cu) (net 9))
-  (segment (start 156.47 126.2) (end 156.47 125.45) (width 0.254) (layer F.Cu) (net 9))
   (segment (start 157.253816 126.562172) (end 157.253816 126.273816) (width 0.254) (layer B.Cu) (net 9))
   (segment (start 157.253816 126.273816) (end 156.47 125.49) (width 0.254) (layer B.Cu) (net 9))
@@
   (segment (start 181.807 132.9) (end 181.864 132.957) (width 0.254) (layer B.Cu) (net 10))
   (segment (start 178.485 132.957) (end 178.179 132.651) (width 0.254) (layer B.Cu) (net 10))
+  (segment (start 208.45 136.49) (end 204.990647 136.49) (width 0.254) (layer F.Cu) (net 11))
+  (segment (start 204.990647 136.49) (end 200.129647 141.351) (width 0.254) (layer F.Cu) (net 11))
+  (segment (start 200.129647 141.351) (end 196.0245 141.351) (width 0.254) (layer F.Cu) (net 11))
+  (segment (start 169.818696 139.22851) (end 169.190079 139.22851) (width 0.254) (layer F.Cu) (net 11))
+  (segment (start 196.0245 141.351) (end 192.5955 144.78) (width 0.254) (layer F.Cu) (net 11))
+  (segment (start 192.5955 144.78) (end 179.51 144.78) (width 0.254) (layer F.Cu) (net 11))
+  (segment (start 179.51 144.78) (end 173.95851 139.22851) (width 0.254) (layer F.Cu) (net 11))
   (segment (start 173.95851 139.22851) (end 169.818696 139.22851) (width 0.254) (layer F.Cu) (net 11))
-  (segment (start 208.45 136.49) (end 204.990647 136.49) (width 0.254) (layer F.Cu) (net 11))
-  (segment (start 196.186636 145.294011) (end 180.024011 145.294011) (width 0.254) (layer F.Cu) (net 11))
-  (segment (start 180.024011 145.294011) (end 173.95851 139.22851) (width 0.254) (layer F.Cu) (net 11))
   (segment (start 169.190079 139.011079) (end 169.190079 139.22851) (width 0.254) (layer B.Cu) (net 11))
-  (segment (start 169.818696 139.22851) (end 169.190079 139.22851) (width 0.254) (layer F.Cu) (net 11))
   (segment (start 163.079 132.9) (end 169.190079 139.011079) (width 0.254) (layer B.Cu) (net 11))
   (segment (start 162.179 132.9) (end 163.079 132.9) (width 0.254) (layer B.Cu) (net 11))
-  (segment (start 204.990647 136.49) (end 196.186636 145.294011) (width 0.254) (layer F.Cu) (net 11))
   (via (at 169.190079 139.22851) (size 0.889) (drill 0.635) (layers F.Cu B.Cu) (net 11))
   (segment (start 178.179 136.9) (end 175.3295 136.9) (width 0.254) (layer B.Cu) (net 12))
@@
   (segment (start 184.658002 138.049) (end 184.467502 138.2395) (width 0.254) (layer B.Cu) (net 14))
   (via (at 184.467502 138.2395) (size 0.889) (drill 0.635) (layers F.Cu B.Cu) (net 14))
-  (segment (start 180.8 144.94) (end 174.417 138.557) (width 0.254) (layer F.Cu) (net 15))
-  (segment (start 174.417 138.557) (end 167.64 138.557) (width 0.254) (layer F.Cu) (net 15))
-  (segment (start 196.04 144.94) (end 180.8 144.94) (width 0.254) (layer F.Cu) (net 15))
-  (segment (start 203.23 137.75) (end 196.04 144.94) (width 0.254) (layer F.Cu) (net 15))
   (segment (start 203.23 130.58) (end 203.23 137.75) (width 0.254) (layer F.Cu) (net 15))
+  (segment (start 203.23 137.75) (end 200.01 140.97) (width 0.254) (layer F.Cu) (net 15))
+  (segment (start 200.01 140.97) (end 195.7705 140.97) (width 0.254) (layer F.Cu) (net 15))
+  (segment (start 174.417 138.557) (end 168.268617 138.557) (width 0.254) (layer F.Cu) (net 15))
+  (segment (start 168.268617 138.557) (end 167.64 138.557) (width 0.254) (layer F.Cu) (net 15))
+  (segment (start 195.7705 140.97) (end 192.314511 144.425989) (width 0.254) (layer F.Cu) (net 15))
+  (segment (start 192.314511 144.425989) (end 180.285989 144.425989) (width 0.254) (layer F.Cu) (net 15))
+  (segment (start 180.285989 144.425989) (end 174.417 138.557) (width 0.254) (layer F.Cu) (net 15))
   (segment (start 167.64 138.557) (end 165.862 138.557) (width 0.254) (layer B.Cu) (net 15))
   (via (at 167.64 138.557) (size 0.889) (drill 0.635) (layers F.Cu B.Cu) (net 15))
@@
   (segment (start 126.8095 138.1705) (end 127.53 137.45) (width 0.254) (layer B.Cu) (net 17))
   (via (at 127.53 137.45) (size 0.889) (drill 0.635) (layers F.Cu B.Cu) (net 17))
-  (segment (start 153.9255 129.0955) (end 159.327883 129.0955) (width 0.254) (layer F.Cu) (net 18))
-  (segment (start 152.775989 127.945989) (end 153.9255 129.0955) (width 0.254) (layer F.Cu) (net 18))
+  (segment (start 126.18 135.56) (end 126.18 133.4) (width 0.254) (layer F.Cu) (net 18))
+  (segment (start 154.9415 130.1115) (end 158.692883 130.1115) (width 0.254) (layer F.Cu) (net 18))
+  (segment (start 126.18 133.4) (end 131.634011 127.945989) (width 0.254) (layer F.Cu) (net 18))
   (segment (start 131.634011 127.945989) (end 152.775989 127.945989) (width 0.254) (layer F.Cu) (net 18))
-  (segment (start 126.18 133.4) (end 131.634011 127.945989) (width 0.254) (layer F.Cu) (net 18))
-  (segment (start 126.18 135.56) (end 126.18 133.4) (width 0.254) (layer F.Cu) (net 18))
-  (segment (start 160.152 128.9) (end 159.9565 129.0955) (width 0.254) (layer B.Cu) (net 18))
-  (segment (start 159.327883 129.0955) (end 159.9565 129.0955) (width 0.254) (layer F.Cu) (net 18))
-  (via (at 159.9565 129.0955) (size 0.889) (drill 0.635) (layers F.Cu B.Cu) (net 18))
-  (segment (start 162.179 128.9) (end 160.152 128.9) (width 0.254) (layer B.Cu) (net 18))
+  (segment (start 152.775989 127.945989) (end 154.9415 130.1115) (width 0.254) (layer F.Cu) (net 18))
+  (segment (start 158.692883 130.1115) (end 159.264383 129.54) (width 0.254) (layer F.Cu) (net 18))
+  (segment (start 159.264383 129.54) (end 159.893 129.54) (width 0.254) (layer F.Cu) (net 18))
+  (segment (start 159.893 129.432) (end 159.893 129.54) (width 0.254) (layer B.Cu) (net 18))
+  (segment (start 160.425 128.9) (end 159.893 129.432) (width 0.254) (layer B.Cu) (net 18))
+  (segment (start 162.179 128.9) (end 160.425 128.9) (width 0.254) (layer B.Cu) (net 18))
+  (via (at 159.893 129.54) (size 0.889) (drill 0.635) (layers F.Cu B.Cu) (net 18))
   (segment (start 125.5395 137.7315) (end 125.476 137.668) (width 0.254) (layer B.Cu) (net 18))
   (segment (start 125.5395 138.938) (end 125.5395 137.7315) (width 0.254) (layer B.Cu) (net 18))
@@
   (via (at 146.25 141.08) (size 0.889) (drill 0.635) (layers F.Cu B.Cu) (net 36))
   (via (at 151.77 137.93) (size 0.889) (drill 0.635) (layers F.Cu B.Cu) (net 36))
+  (segment (start 212.09 130.302) (end 212.09 135.91) (width 0.3048) (layer F.Cu) (net 37))
+  (segment (start 212.09 135.91) (end 206.2045 141.7955) (width 0.3048) (layer F.Cu) (net 37))
+  (segment (start 206.2045 141.7955) (end 196.215 141.7955) (width 0.3048) (layer F.Cu) (net 37))
+  (segment (start 150.761604 139.925412) (end 150.161515 140.525501) (width 0.3048) (layer F.Cu) (net 37))
+  (segment (start 196.215 141.7955) (end 192.8495 145.161) (width 0.3048) (layer F.Cu) (net 37))
+  (segment (start 192.8495 145.161) (end 178.624432 145.161) (width 0.3048) (layer F.Cu) (net 37))
+  (segment (start 178.624432 145.161) (end 173.388844 139.925412) (width 0.3048) (layer F.Cu) (net 37))
+  (segment (start 173.388844 139.925412) (end 150.761604 139.925412) (width 0.3048) (layer F.Cu) (net 37))
+  (segment (start 150.161515 140.525501) (end 149.717016 140.97) (width 0.3048) (layer F.Cu) (net 37))
   (segment (start 149.717016 141.517984) (end 149.717016 140.97) (width 0.3048) (layer B.Cu) (net 37))
   (segment (start 148.855 142.38) (end 149.717016 141.517984) (width 0.3048) (layer B.Cu) (net 37))
-  (segment (start 212.09 135.91) (end 202.32658 145.67342) (width 0.3048) (layer F.Cu) (net 37))
   (segment (start 148.22 142.38) (end 148.855 142.38) (width 0.3048) (layer B.Cu) (net 37))
-  (segment (start 150.161515 140.525501) (end 149.717016 140.97) (width 0.3048) (layer F.Cu) (net 37))
-  (segment (start 173.388844 139.925412) (end 150.761604 139.925412) (width 0.3048) (layer F.Cu) (net 37))
-  (segment (start 150.761604 139.925412) (end 150.161515 140.525501) (width 0.3048) (layer F.Cu) (net 37))
-  (segment (start 179.136852 145.67342) (end 173.388844 139.925412) (width 0.3048) (layer F.Cu) (net 37))
-  (segment (start 202.32658 145.67342) (end 179.136852 145.67342) (width 0.3048) (layer F.Cu) (net 37))
-  (segment (start 212.09 130.302) (end 212.09 135.91) (width 0.3048) (layer F.Cu) (net 37))
   (via (at 149.717016 140.97) (size 0.889) (drill 0.635) (layers F.Cu B.Cu) (net 37))
   (segment (start 156.62 141.24) (end 157.034501 141.654501) (width 0.254) (layer B.Cu) (net 38))
@@
     (polygon
       (pts
-        (xy 159.766 120.523) (xy 159.766 127.508) (xy 180.975 127.508) (xy 180.975 120.523)
+        (xy 159.766 120.523) (xy 159.766 127.127) (xy 180.975 127.127) (xy 180.975 120.523)
       )
     )
