File: Sensors.sch (KiCad schematic (older format))
At the start: 13 parts, among them Q3 S8050, SW1 COLLISION, SW2 COLLISION, U1 phototransistor, U2 phototransistor, U3 PCF8591

Commit message: v3.2 of the PCB
Parts:
- removed Q3: S8050, Custom:SOT-23, symbol S8050
- removed R13: 10k, Resistors_SMD:R_0603, symbol R
- removed R9: 160R, Resistors_SMD:R_0603, symbol R
Connections:
- net LED_EN: now also D2.1 (K)
- net at D1.1 (K): now also D2.2 (A); no longer D2.1 (K)
Other:
- moved on the sheet: D1, D2, R7, R8, U2

Commit message: v3.5 of the PCB
Parts:
- D1, D2: Manfr. Part Number (MFP) (none) -> KPA3010F3C; Manufacturer Name (MFN) (none) -> Kingbright; Package ID (none) -> 0603
- U1, U2: Manfr. Part Number (MFP) (none) -> KPA-3010P3C; Manufacturer Name (MFN) (none) -> Kingbright; Package ID (none) -> 0603
- U3: Source2 http://www.aliexpress.com/item/20pcs-lot-PCF8591T/324041985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 -> (none); http://www.aliexpress.com/item/20pcs-lot-PCF8591T/32404198526.html (none) -> =HYPERLINK(
Changed lines of the file:
@@
 F 6 "NXP" H 6775 4100 60  0001 C CNN "Manufacturer Name (MFN)"
 F 7 "PCF8591T" H 6775 4100 60  0001 C CNN "Manfr. Part Number (MFP)"
-F 8 "http://www.aliexpress.com/item/20pcs-lot-PCF8591T/32404198526.html" H 6775 4100 60  0001 C CNN "Source2"
+F 8 "=HYPERLINK(" H 0   0   60  0001 C CNN "http://www.aliexpress.com/item/20pcs-lot-PCF8591T/32404198526.html"
 F 9 "y" H 6775 4100 60  0001 C CNN "Required"
 	1    6775 4100
@@
 NoConn ~ 7525 3700
 $Comp
-L +3V3 #PWR012
+L +3V3 #PWR014
 U 1 1 569FF9A4
 P 6775 3200
-F 0 "#PWR012" H 6775 3050 60  0001 C CNN
+F 0 "#PWR014" H 6775 3050 60  0001 C CNN
 F 1 "+3V3" H 6775 3340 60  0000 C CNN
 F 2 "" H 6775 3200 60  0000 C CNN
@@
 $EndComp
 $Comp
-L GND #PWR013
+L GND #PWR015
 U 1 1 569FF9AA
 P 6775 5000
-F 0 "#PWR013" H 6775 4750 60  0001 C CNN
+F 0 "#PWR015" H 6775 4750 60  0001 C CNN
 F 1 "GND" H 6775 4850 60  0000 C CNN
 F 2 "" H 6775 5000 60  0000 C CNN
@@
 NoConn ~ 7450 4500
 $Comp
-L +3V3 #PWR014
+L +3V3 #PWR016
 U 1 1 569FF9BE
 P 7575 3925
-F 0 "#PWR014" H 7575 3775 60  0001 C CNN
+F 0 "#PWR016" H 7575 3775 60  0001 C CNN
 F 1 "+3V3" H 7575 4065 60  0000 C CNN
 F 2 "" H 7575 3925 60  0000 C CNN
@@
 F 1 "phototransistor" H 4450 2300 60  0000 C CNN
 F 2 "Custom:SIDE-LED" H 4450 2000 60  0001 C CNN
-F 3 "" H 4450 2000 60  0000 C CNN
+F 3 "=HYPERLINK(\"\"http://webtest4.kingbright.com/attachments/file/psearch/000/00/00/KPA-3010P3C(Ver.16).pdf\"\", \"\"[LINK]\"\")" H 4450 2000 60  0001 C CNN
 F 4 "Side facing SMD infrared phototransistor" H 4450 2000 60  0001 C CNN "Description"
-F 5 "y" H 4450 2000 60  0001 C CNN "Required"
+F 5 "0603" H 4450 2000 60  0001 C CNN "Package ID"
+F 6 "Kingbright" H 4450 2000 60  0001 C CNN "Manufacturer Name (MFN)"
+F 7 "KPA-3010P3C" H 4450 2000 60  0001 C CNN "Manfr. Part Number (MFP)"
+F 8 "y" H 4450 2000 60  0001 C CNN "Required"
 	1    4450 2000
 	-1   0    0    -1
@@
 F 1 "LED" H 4450 1225 50  0000 C CNN
 F 2 "Custom:SIDE-LED-REVERSED" H 4450 1325 50  0001 C CNN
-F 3 "" H 4450 1325 50  0000 C CNN
+F 3 "=HYPERLINK(\"\"www.kingbright.com/attachments/file/psearch/000/00/20131112/KPA-3010F3C(Ver.15A).pdf\"\", \"\"[link]\"\")" H 4450 1325 60  0001 C CNN
 F 4 "Side facing SMD infrared LED" H 4450 1325 60  0001 C CNN "Description"
-F 5 "y" H 4450 1325 60  0001 C CNN "Required"
+F 5 "0603" H 4450 1325 60  0001 C CNN "Package ID"
+F 6 "Kingbright" H 4450 1325 60  0001 C CNN "Manufacturer Name (MFN)"
+F 7 "KPA3010F3C" H 4450 1325 60  0001 C CNN "Manfr. Part Number (MFP)"
+F 8 "y" H 4450 1325 60  0001 C CNN "Required"
 	1    4450 1325
 	-1   0    0    1
@@
 F 1 "phototransistor" H 6275 2300 60  0000 C CNN
 F 2 "Custom:SIDE-LED" H 6275 2000 60  0001 C CNN
-F 3 "" H 6275 2000 60  0000 C CNN
-F 4 "Side facing SMD infrared phototransistor" H 6275 2000 60  0001 C CNN "Description"
-F 5 "y" H 6275 2000 60  0001 C CNN "Required"
+F 3 "=HYPERLINK(\"\"http://webtest4.kingbright.com/attachments/file/psearch/000/00/00/KPA-3010P3C(Ver.16).pdf\"\", \"\"[LINK]\"\")" H 4450 2000 60  0001 C CNN
+F 4 "Side facing SMD infrared phototransistor" H 4450 2000 60  0001 C CNN "Description"
+F 5 "0603" H 4450 2000 60  0001 C CNN "Package ID"
+F 6 "Kingbright" H 4450 2000 60  0001 C CNN "Manufacturer Name (MFN)"
+F 7 "KPA-3010P3C" H 4450 2000 60  0001 C CNN "Manfr. Part Number (MFP)"
+F 8 "y" H 4450 2000 60  0001 C CNN "Required"
 	1    6275 2000
 	-1   0    0    -1
@@
 F 1 "LED" H 6275 1225 50  0000 C CNN
 F 2 "Custom:SIDE-LED-REVERSED" H 6275 1325 50  0001 C CNN
-F 3 "" H 6275 1325 50  0000 C CNN
-F 4 "Side facing SMD infrared LED" H 6275 1325 60  0001 C CNN "Description"
-F 5 "y" H 6275 1325 60  0001 C CNN "Required"
+F 3 "=HYPERLINK(" H 6275 1325 60  0001 C CNN
+F 4 "Side facing SMD infrared LED" H 4450 1325 60  0001 C CNN "Description"
+F 5 "0603" H 4450 1325 60  0001 C CNN "Package ID"
+F 6 "Kingbright" H 4450 1325 60  0001 C CNN "Manufacturer Name (MFN)"
+F 7 "KPA3010F3C" H 4450 1325 60  0001 C CNN "Manfr. Part Number (MFP)"
+F 8 "y" H 4450 1325 60  0001 C CNN "Required"
 	1    6275 1325
 	-1   0    0    1
 $EndComp
 $Comp
-L +3V3 #PWR015
+L +3V3 #PWR017
 U 1 1 569FFA18
 P 3450 1075
-F 0 "#PWR015" H 3450 925 60  0001 C CNN
+F 0 "#PWR017" H 3450 925 60  0001 C CNN
 F 1 "+3V3" H 3450 1215 60  0000 C CNN
 F 2 "" H 3450 1075 60  0000 C CNN
@@
 F 1 "COLLISION" H 4315 4775 59  0000 C CNN
 F 2 "Custom:LEVER_SWITCH" H 4275 5025 60  0001 C CNN
-F 3 "" H 4275 5025 60  0000 C CNN
+F 3 "=HYPERLINK(\"\"https://www.aliexpress.com/item/Lever-Button-Micro-Switch-long-lever/1888268351.html\"\", \"\"[LINK]\"\")" H 4275 5025 60  0001 C CNN
 F 4 "Long lever switch" H 4275 5025 60  0001 C CNN "Description"
 F 5 "y" H 4275 5025 60  0001 C CNN "Required"
@@
 F 1 "COLLISION" H 4315 4075 59  0000 C CNN
 F 2 "Custom:LEVER_SWITCH" H 4275 4325 60  0001 C CNN
-F 3 "" H 4275 4325 60  0000 C CNN
+F 3 "=HYPERLINK(\"\"https://www.aliexpress.com/item/Lever-Button-Micro-Switch-long-lever/1888268351.html\"\", \"\"[LINK]\"\")" H 4275 4325 60  0001 C CNN
 F 4 "Long lever switch" H 4275 5025 60  0001 C CNN "Description"
 F 5 "y" H 4275 5025 60  0001 C CNN "Required"
@@
 $EndComp
 $Comp
-L GND #PWR016
+L GND #PWR018
 U 1 1 56A5FE25
 P 3750 5275
-F 0 "#PWR016" H 3750 5025 60  0001 C CNN
+F 0 "#PWR018" H 3750 5025 60  0001 C CNN
 F 1 "GND" H 3750 5125 60  0000 C CNN
 F 2 "" H 3750 5275 60  0000 C CNN
@@
 $EndComp
 $Comp
-L +3V3 #PWR017
+L +3V3 #PWR019
 U 1 1 56A6005C
 P 3625 3925
-F 0 "#PWR017" H 3625 3775 60  0001 C CNN
+F 0 "#PWR019" H 3625 3775 60  0001 C CNN
 F 1 "+3V3" H 3625 4065 60  0000 C CNN
 F 2 "" H 3625 3925 60  0000 C CNN
@@
 $EndComp
 $Comp
-L GND #PWR018
+L GND #PWR020
 U 1 1 56B4B00B
 P 7450 2200
-F 0 "#PWR018" H 7450 1950 60  0001 C CNN
+F 0 "#PWR020" H 7450 1950 60  0001 C CNN
 F 1 "GND" H 7450 2050 60  0000 C CNN
 F 2 "" H 7450 2200 60  0000 C CNN
@@
 NoConn ~ 4675 5225
 $Comp
-L +3V3 #PWR019
+L +3V3 #PWR021
 U 1 1 56D9B5C7
 P 5275 1800
-F 0 "#PWR019" H 5275 1650 60  0001 C CNN
+F 0 "#PWR021" H 5275 1650 60  0001 C CNN
 F 1 "+3V3" H 5275 1940 60  0000 C CNN
 F 2 "" H 5275 1800 60  0000 C CNN
@@
 $EndComp
 $Comp
-L GND #PWR020
+L GND #PWR022
 U 1 1 56D9B9AB
 P 4800 2200
-F 0 "#PWR020" H 4800 1950 60  0001 C CNN
+F 0 "#PWR022" H 4800 1950 60  0001 C CNN
 F 1 "GND" H 4800 2050 60  0000 C CNN
 F 2 "" H 4800 2200 60  0000 C CNN

Commit message: v3.6 of the PCB
Parts:
- SW1, SW2: Description Long lever switch -> 23mm Long lever switch
- U3: Source1 (none) -> http://www.aliexpress.com/item/20pcs-lot-PCF8591T/324041985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; http://www.aliexpress.com/item/20pcs-lot-PCF8591T/32404198526.html =HYPERLINK( -> (none)
Changed lines of the file:
@@
 F 6 "NXP" H 6775 4100 60  0001 C CNN "Manufacturer Name (MFN)"
 F 7 "PCF8591T" H 6775 4100 60  0001 C CNN "Manfr. Part Number (MFP)"
-F 8 "=HYPERLINK(" H 0   0   60  0001 C CNN "http://www.aliexpress.com/item/20pcs-lot-PCF8591T/32404198526.html"
+F 8 "http://www.aliexpress.com/item/20pcs-lot-PCF8591T/32404198526.html" H 0   0   60  0001 C CNN "Source1"
 F 9 "y" H 6775 4100 60  0001 C CNN "Required"
 	1    6775 4100
@@
 F 1 "phototransistor" H 4450 2300 60  0000 C CNN
 F 2 "Custom:SIDE-LED" H 4450 2000 60  0001 C CNN
-F 3 "=HYPERLINK(\"\"http://webtest4.kingbright.com/attachments/file/psearch/000/00/00/KPA-3010P3C(Ver.16).pdf\"\", \"\"[LINK]\"\")" H 4450 2000 60  0001 C CNN
+F 3 "http://webtest4.kingbright.com/attachments/file/psearch/000/00/00/KPA-3010P3C(Ver.16).pdf" H 4450 2000 60  0001 C CNN
 F 4 "Side facing SMD infrared phototransistor" H 4450 2000 60  0001 C CNN "Description"
 F 5 "0603" H 4450 2000 60  0001 C CNN "Package ID"
@@
 F 1 "LED" H 4450 1225 50  0000 C CNN
 F 2 "Custom:SIDE-LED-REVERSED" H 4450 1325 50  0001 C CNN
-F 3 "=HYPERLINK(\"\"www.kingbright.com/attachments/file/psearch/000/00/20131112/KPA-3010F3C(Ver.15A).pdf\"\", \"\"[link]\"\")" H 4450 1325 60  0001 C CNN
+F 3 "http://www.kingbright.com/attachments/file/psearch/000/00/20131112/KPA-3010F3C(Ver.15A).pdf" H 4450 1325 60  0001 C CNN
 F 4 "Side facing SMD infrared LED" H 4450 1325 60  0001 C CNN "Description"
 F 5 "0603" H 4450 1325 60  0001 C CNN "Package ID"
@@
 F 1 "phototransistor" H 6275 2300 60  0000 C CNN
 F 2 "Custom:SIDE-LED" H 6275 2000 60  0001 C CNN
-F 3 "=HYPERLINK(\"\"http://webtest4.kingbright.com/attachments/file/psearch/000/00/00/KPA-3010P3C(Ver.16).pdf\"\", \"\"[LINK]\"\")" H 4450 2000 60  0001 C CNN
+F 3 "http://webtest4.kingbright.com/attachments/file/psearch/000/00/00/KPA-3010P3C(Ver.16).pdf" H 4450 2000 60  0001 C CNN
 F 4 "Side facing SMD infrared phototransistor" H 4450 2000 60  0001 C CNN "Description"
 F 5 "0603" H 4450 2000 60  0001 C CNN "Package ID"
@@
 F 1 "COLLISION" H 4315 4775 59  0000 C CNN
 F 2 "Custom:LEVER_SWITCH" H 4275 5025 60  0001 C CNN
-F 3 "=HYPERLINK(\"\"https://www.aliexpress.com/item/Lever-Button-Micro-Switch-long-lever/1888268351.html\"\", \"\"[LINK]\"\")" H 4275 5025 60  0001 C CNN
-F 4 "Long lever switch" H 4275 5025 60  0001 C CNN "Description"
+F 3 "https://www.aliexpress.com/item/Lever-Button-Micro-Switch-long-lever/1888268351.html" H 4275 5025 60  0001 C CNN
+F 4 "23mm Long lever switch" H 4275 5025 60  0001 C CNN "Description"
 F 5 "y" H 4275 5025 60  0001 C CNN "Required"
 	1    4275 5025
@@
 F 1 "COLLISION" H 4315 4075 59  0000 C CNN
 F 2 "Custom:LEVER_SWITCH" H 4275 4325 60  0001 C CNN
-F 3 "=HYPERLINK(\"\"https://www.aliexpress.com/item/Lever-Button-Micro-Switch-long-lever/1888268351.html\"\", \"\"[LINK]\"\")" H 4275 4325 60  0001 C CNN
-F 4 "Long lever switch" H 4275 5025 60  0001 C CNN "Description"
+F 3 "https://www.aliexpress.com/item/Lever-Button-Micro-Switch-long-lever/1888268351.html" H 4275 4325 60  0001 C CNN
+F 4 "23mm Long lever switch" H 4275 5025 60  0001 C CNN "Description"
 F 5 "y" H 4275 5025 60  0001 C CNN "Required"
 	1    4275 4325
