File: power.sch (KiCad schematic (older format))
At the start: 8 parts, among them SW3 POWER_SWITCH, U8 LD1117S33CTR

Commit message: v3.3 of the PCB
Parts:
- BATT1: footprint Pin_Headers:Pin_Header_Straight_1x02 -> Custom:JST_XH-1x02
Changed lines of the file:
@@
 F 0 "BATT1" H 2775 3475 50  0000 C CNN
 F 1 "BATT" V 2875 3325 50  0000 C CNN
-F 2 "Pin_Headers:Pin_Header_Straight_1x02" H 2775 3325 60  0001 C CNN
+F 2 "Custom:JST_XH-1x02" H 2775 3325 60  0001 C CNN
 F 3 "http://www.jst-mfg.com/product/pdf/eng/eXH.pdf" H 2775 3325 60  0001 C CNN
 F 4 "JST XH 2 Pin Male Socket" H 2775 3325 60  0001 C CNN "Description"
@@
 $EndComp
 $Comp
-L GND #PWR034
+L GND #PWR032
 U 1 1 56A07466
 P 3175 3550
-F 0 "#PWR034" H 3175 3300 60  0001 C CNN
+F 0 "#PWR032" H 3175 3300 60  0001 C CNN
 F 1 "GND" H 3175 3400 60  0000 C CNN
 F 2 "" H 3175 3550 60  0000 C CNN
@@
 $EndComp
 $Comp
-L VSS #PWR035
+L VSS #PWR033
 U 1 1 56A0746C
 P 5200 2925
-F 0 "#PWR035" H 5200 2775 60  0001 C CNN
+F 0 "#PWR033" H 5200 2775 60  0001 C CNN
 F 1 "VSS" H 5200 3075 60  0000 C CNN
 F 2 "" H 5200 2925 60  0000 C CNN
@@
 $EndComp
 $Comp
-L PWR_FLAG #FLG036
+L PWR_FLAG #FLG034
 U 1 1 56A07CE8
 P 3950 6375
-F 0 "#FLG036" H 3950 6470 30  0001 C CNN
+F 0 "#FLG034" H 3950 6470 30  0001 C CNN
 F 1 "PWR_FLAG" H 3950 6555 30  0000 C CNN
 F 2 "" H 3950 6375 60  0000 C CNN
@@
 $EndComp
 $Comp
-L PWR_FLAG #FLG037
+L PWR_FLAG #FLG035
 U 1 1 56A07CEE
 P 4350 6375
-F 0 "#FLG037" H 4350 6470 30  0001 C CNN
+F 0 "#FLG035" H 4350 6470 30  0001 C CNN
 F 1 "PWR_FLAG" H 4350 6555 30  0000 C CNN
 F 2 "" H 4350 6375 60  0000 C CNN
@@
 $EndComp
 $Comp
-L PWR_FLAG #FLG038
+L PWR_FLAG #FLG036
 U 1 1 56A07CF4
 P 4750 6375
-F 0 "#FLG038" H 4750 6470 30  0001 C CNN
+F 0 "#FLG036" H 4750 6470 30  0001 C CNN
 F 1 "PWR_FLAG" H 4750 6555 30  0000 C CNN
 F 2 "" H 4750 6375 60  0000 C CNN
@@
 $EndComp
 $Comp
-L GND #PWR039
+L GND #PWR037
 U 1 1 56A07CFA
 P 4750 6550
-F 0 "#PWR039" H 4750 6300 60  0001 C CNN
+F 0 "#PWR037" H 4750 6300 60  0001 C CNN
 F 1 "GND" H 4750 6400 60  0000 C CNN
 F 2 "" H 4750 6550 60  0000 C CNN
@@
 $EndComp
 $Comp
-L VSS #PWR040
+L VSS #PWR038
 U 1 1 56A07D00
 P 4350 6550
-F 0 "#PWR040" H 4350 6400 60  0001 C CNN
+F 0 "#PWR038" H 4350 6400 60  0001 C CNN
 F 1 "VSS" H 4350 6700 60  0000 C CNN
 F 2 "" H 4350 6550 60  0000 C CNN
@@
 $EndComp
 $Comp
-L +3V3 #PWR041
+L +3V3 #PWR039
 U 1 1 56A07D06
 P 3950 6550
-F 0 "#PWR041" H 3950 6400 60  0001 C CNN
+F 0 "#PWR039" H 3950 6400 60  0001 C CNN
 F 1 "+3V3" H 3950 6690 60  0000 C CNN
 F 2 "" H 3950 6550 60  0000 C CNN
@@
 $EndComp
 $Comp
-L GND #PWR042
+L GND #PWR040
 U 1 1 56A083CE
 P 6200 3800
-F 0 "#PWR042" H 6200 3550 60  0001 C CNN
+F 0 "#PWR040" H 6200 3550 60  0001 C CNN
 F 1 "GND" H 6200 3650 60  0000 C CNN
 F 2 "" H 6200 3800 60  0000 C CNN
@@
 $EndComp
 $Comp
-L +3V3 #PWR043
+L +3V3 #PWR041
 U 1 1 56A0851B
 P 7400 2875
-F 0 "#PWR043" H 7400 2725 60  0001 C CNN
+F 0 "#PWR041" H 7400 2725 60  0001 C CNN
 F 1 "+3V3" H 7400 3015 60  0000 C CNN
 F 2 "" H 7400 2875 60  0000 C CNN
@@
 $EndComp
 $Comp
-L VSS #PWR044
+L VSS #PWR042
 U 1 1 56A07D18
 P 2275 6025
-F 0 "#PWR044" H 2275 5875 60  0001 C CNN
+F 0 "#PWR042" H 2275 5875 60  0001 C CNN
 F 1 "VSS" H 2275 6175 60  0000 C CNN
 F 2 "" H 2275 6025 60  0000 C CNN
@@
 $EndComp
 $Comp
-L GND #PWR045
+L GND #PWR043
 U 1 1 56A07D0C
 P 2275 6700
-F 0 "#PWR045" H 2275 6450 60  0001 C CNN
+F 0 "#PWR043" H 2275 6450 60  0001 C CNN
 F 1 "GND" H 2275 6550 60  0000 C CNN
 F 2 "" H 2275 6700 60  0000 C CNN
@@
 	3175 3075 3175 2850
 $Comp
-L +5V #PWR046
+L +5V #PWR044
 U 1 1 56B2F9C1
 P 3175 2850
-F 0 "#PWR046" H 3175 2700 60  0001 C CNN
+F 0 "#PWR044" H 3175 2700 60  0001 C CNN
 F 1 "+5V" H 3175 2990 60  0000 C CNN
 F 2 "" H 3175 2850 60  0000 C CNN
@@
 	4425 3175 4225 3175
 $Comp
-L GND #PWR047
+L GND #PWR045
 U 1 1 56B3E3A0
 P 4300 3550
-F 0 "#PWR047" H 4300 3300 60  0001 C CNN
+F 0 "#PWR045" H 4300 3300 60  0001 C CNN
 F 1 "GND" H 4300 3400 60  0000 C CNN
 F 2 "" H 4300 3550 60  0000 C CNN

Commit message: v3.5 of the PCB
Parts:
- removed BATT1: BATT, Custom:JST_XH-1x02, symbol CONN_01X02
- added BATT1: BATT, Connectors_JST:JST_PH_B3B-PH-K_03x2.00mm_Straight, symbol CONN_01X03
- added W7, W8: TEST_1P, Measurement_Points:Measurement_Point_Round-SMD-Pad_Small, symbol TEST_1P
Connections:
- net +5V: now also SW3.1, BATT1.2 (P2); no longer SW3.3
- net GND: now also BATT1.1 (P1), W7.1
- net at F1.1, SW3.2: now also W8.1
- new net: BATT1.3 (P3), SW3.3
Changed lines of the file:
@@
 $EndDescr
-$Comp
-L CONN_01X02 BATT1
-U 1 1 56A0745F
-P 2775 3325
-F 0 "BATT1" H 2775 3475 50  0000 C CNN
-F 1 "BATT" V 2875 3325 50  0000 C CNN
-F 2 "Custom:JST_XH-1x02" H 2775 3325 60  0001 C CNN
-F 3 "http://www.jst-mfg.com/product/pdf/eng/eXH.pdf" H 2775 3325 60  0001 C CNN
-F 4 "JST XH 2 Pin Male Socket" H 2775 3325 60  0001 C CNN "Description"
-F 5 "JST" H 2775 3325 60  0001 C CNN "Manufacturer Name (MFN)"
-F 6 "B2B-XH-A" H 2775 3325 60  0001 C CNN "Manfr. Part Number (MFP)"
-F 7 "http://www.digikey.co.uk/product-detail/en/B2B-XH-A(LF)(SN)/455-2247-ND/1651045" H 2775 3325 60  0001 C CNN "Source1"
-F 8 "y" H 2775 3325 60  0001 C CNN "Required"
-	1    2775 3325
-	-1   0    0    1
-$EndComp
 $Comp
 L GND #PWR032
@@
 F 1 "POWER_SWITCH" H 3865 2925 59  0000 C CNN
 F 2 "Custom:SMALL_SLIDE_SWITCH" H 3825 3175 60  0001 C CNN
-F 3 "" H 3825 3175 60  0000 C CNN
+F 3 "=HYPERLINK(\"\"https://www.aliexpress.com/item/10Pcs-Toggle-switch-SK12D07VG3-stents-Small-toggle-switch-3-mm-high-Miniature-Slide-Switch-Side-Knob/32762894678.html\"\",\"\"[LINK]\"\")" H 3825 3175 60  0001 C CNN
 F 4 "SPDT Slide Switch R/A" H 3825 3175 60  0001 C CNN "Description"
 F 5 "Generic" H 3825 3175 60  0001 C CNN "Manufacturer Name (MFN)"
@@
 	1    0    0    -1
 $EndComp
-Wire Wire Line
-	4925 3175 5800 3175
-Wire Wire Line
-	3425 3275 2975 3275
-Wire Wire Line
-	2975 3375 3175 3375
-Wire Wire Line
-	3175 3375 3175 3550
-Wire Wire Line
-	5200 3175 5200 2925
-Wire Wire Line
-	4750 6375 4750 6550
-Wire Wire Line
-	4350 6375 4350 6550
-Wire Wire Line
-	3950 6375 3950 6550
-Connection ~ 5200 3175
-Wire Wire Line
-	6200 3475 6200 3800
-Wire Wire Line
-	6600 3175 7400 3175
-Wire Wire Line
-	7400 3175 7400 2875
-Wire Wire Line
-	5575 3275 5575 3175
-Connection ~ 5575 3175
-Wire Wire Line
-	6725 3275 6725 3175
-Connection ~ 6725 3175
-Wire Wire Line
-	7075 3275 7075 3175
-Connection ~ 7075 3175
-Wire Wire Line
-	5575 3575 5575 3700
-Wire Wire Line
-	5575 3700 7075 3700
-Connection ~ 6200 3700
-Wire Wire Line
-	7075 3700 7075 3575
-Wire Wire Line
-	6725 3575 6725 3700
-Connection ~ 6725 3700
-Wire Wire Line
-	2275 6500 2275 6700
-Wire Wire Line
-	2275 6200 2275 6025
 $Comp
 L CP1 C1
@@
 	1    0    0    -1
 $EndComp
-Wire Wire Line
-	3425 3075 3175 3075
-Wire Wire Line
-	3175 3075 3175 2850
 $Comp
 L +5V #PWR044
@@
 	1    0    0    -1
 $EndComp
-Wire Wire Line
-	4425 3175 4225 3175
 $Comp
 L GND #PWR045
@@
 	1    0    0    -1
 $EndComp
+$Comp
+L CONN_01X03 BATT1
+U 1 1 59B7F792
+P 2775 3175
+F 0 "BATT1" H 2775 3375 50  0000 C CNN
+F 1 "BATT" V 2875 3175 50  0000 C CNN
+F 2 "Connectors_JST:JST_PH_B3B-PH-K_03x2.00mm_Straight" H 2775 3175 50  0001 C CNN
+F 3 "" H 2775 3175 50  0000 C CNN
+	1    2775 3175
+	-1   0    0    1
+$EndComp
+Wire Wire Line
+	3175 3275 2975 3275
+Wire Wire Line
+	3175 3550 3175 3275
+Wire Wire Line
+	4300 3375 4300 3550
 Wire Wire Line
 	4225 3375 4300 3375
 Wire Wire Line
-	4300 3375 4300 3550
+	4425 3175 4225 3175
+Wire Wire Line
+	2275 6200 2275 6025
+Wire Wire Line
+	2275 6500 2275 6700
+Connection ~ 6725 3700
+Wire Wire Line
+	6725 3575 6725 3700
+Wire Wire Line
+	7075 3700 7075 3575
+Connection ~ 6200 3700
+Wire Wire Line
+	5575 3700 7075 3700
+Wire Wire Line
+	5575 3575 5575 3700
+Connection ~ 7075 3175
+Wire Wire Line
+	7075 3275 7075 3175
+Connection ~ 6725 3175
+Wire Wire Line
+	6725 3275 6725 3175
+Connection ~ 5575 3175
+Wire Wire Line
+	5575 3275 5575 3175
+Wire Wire Line
+	7400 3175 7400 2875
+Wire Wire Line
+	6600 3175 7400 3175
+Wire Wire Line
+	6200 3475 6200 3800
+Connection ~ 5200 3175
+Wire Wire Line
+	3950 6375 3950 6550
+Wire Wire Line
+	4350 6375 4350 6550
+Wire Wire Line
+	4750 6375 4750 6550
+Wire Wire Line
+	5200 3175 5200 2925
+Wire Wire Line
+	4925 3175 5800 3175
+Wire Wire Line
+	3425 3275 3425 3175
+Wire Wire Line
+	3425 3175 2975 3175
+Wire Wire Line
+	3175 2850 3175 3175
+Connection ~ 3175 3175
+Wire Wire Line
+	3425 3075 2975 3075
+$Comp
+L TEST_1P W8
+U 1 1 59B82FDC
+P 4325 2975
+F 0 "W8" H 4325 3245 50  0000 C CNN
+F 1 "TEST_1P" H 4325 3175 50  0000 C CNN
+F 2 "Measurement_Points:Measurement_Point_Round-SMD-Pad_Small" H 4525 2975 50  0001 C CNN
+F 3 "" H 4525 2975 50  0000 C CNN
+	1    4325 2975
+	1    0    0    -1
+$EndComp
+Wire Wire Line
+	4325 2975 4325 3175
+Connection ~ 4325 3175
+$Comp
+L TEST_1P W7
+U 1 1 59B831D2
+P 1725 6200
+F 0 "W7" H 1725 6470 50  0000 C CNN
+F 1 "TEST_1P" H 1725 6400 50  0000 C CNN
+F 2 "Measurement_Points:Measurement_Point_Round-SMD-Pad_Small" H 1925 6200 50  0001 C CNN
+F 3 "" H 1925 6200 50  0000 C CNN
+	1    1725 6200
+	1    0    0    -1
+$EndComp
+$Comp
+L GND #PWR046
+U 1 1 59B83226
+P 1725 6425
+F 0 "#PWR046" H 1725 6175 60  0001 C CNN
+F 1 "GND" H 1725 6275 60  0000 C CNN
+F 2 "" H 1725 6425 60  0000 C CNN
+F 3 "" H 1725 6425 60  0000 C CNN
+	1    1725 6425
+	1    0    0    -1
+$EndComp
+Wire Wire Line
+	1725 6200 1725 6425
 $EndSCHEMATC

Commit message: v3.6 of the PCB
Parts:
- BATT1: Description (none) -> JST 3 Pin Through Hole Top entry shrouded header socket; Manfr. Part Number (MFP) (none) -> B3B-PH-K-S; Manufacturer Name (MFN) (none) -> JST; Required (none) -> y
- W8: Required (none) -> n
Changed lines of the file:
@@
 F 1 "POWER_SWITCH" H 3865 2925 59  0000 C CNN
 F 2 "Custom:SMALL_SLIDE_SWITCH" H 3825 3175 60  0001 C CNN
-F 3 "=HYPERLINK(\"\"https://www.aliexpress.com/item/10Pcs-Toggle-switch-SK12D07VG3-stents-Small-toggle-switch-3-mm-high-Miniature-Slide-Switch-Side-Knob/32762894678.html\"\",\"\"[LINK]\"\")" H 3825 3175 60  0001 C CNN
+F 3 "https://www.aliexpress.com/item/10Pcs-Toggle-switch-SK12D07VG3-stents-Small-toggle-switch-3-mm-high-Miniature-Slide-Switch-Side-Knob/32762894678.html" H 3825 3175 60  0001 C CNN
 F 4 "SPDT Slide Switch R/A" H 3825 3175 60  0001 C CNN "Description"
 F 5 "Generic" H 3825 3175 60  0001 C CNN "Manufacturer Name (MFN)"
@@
 F 1 "BATT" V 2875 3175 50  0000 C CNN
 F 2 "Connectors_JST:JST_PH_B3B-PH-K_03x2.00mm_Straight" H 2775 3175 50  0001 C CNN
-F 3 "" H 2775 3175 50  0000 C CNN
+F 3 "http://www.jst-mfg.com/product/pdf/eng/ePH.pdf" H 2775 3175 50  0000 C CNN
+F 4 "JST 3 Pin  Through Hole Top entry shrouded header socket" H 2775 3175 60  0001 C CNN "Description"
+F 5 "JST" H 2775 3175 60  0001 C CNN "Manufacturer Name (MFN)"
+F 6 "B3B-PH-K-S" H 2775 3175 60  0001 C CNN "Manfr. Part Number (MFP)"
+F 7 "y" H 2775 3175 60  0001 C CNN "Required"
 	1    2775 3175
 	-1   0    0    1
@@
 F 2 "Measurement_Points:Measurement_Point_Round-SMD-Pad_Small" H 4525 2975 50  0001 C CNN
 F 3 "" H 4525 2975 50  0000 C CNN
+F 4 "n" H 4325 2975 60  0001 C CNN "Required"
 	1    4325 2975
 	1    0    0    -1
