File: Main/power.sch (KiCad schematic (older format))
At the start: 9 parts, among them SW3 POWER_SWITCH, U8 LD1117S33CTR

Commit message: initial version of v3.0
Parts:
- removed C4: 470uF, Capacitors_SMD:c_elec_8x10, symbol CP2
- removed C5: 100uF, Capacitors_Tantalum_SMD:TantalC_SizeB_EIA-3528_Reflow, symbol CP2
- C6, C8: footprint (none) -> Capacitors_SMD:C_0805
- C7: footprint (none) -> Capacitors_Tantalum_SMD:TantalC_SizeB_EIA-3528_Reflow
- U8: footprint SOT-223 -> TO_SOT_Packages_SMD:SOT-223
Changed lines of the file:
@@
 EESchema Schematic File Version 2
-LIBS:Mirobot-rescue
 LIBS:power
 LIBS:device
@@
 LIBS:memory
 LIBS:xilinx
-LIBS:microcontrollers
-LIBS:dsp
-LIBS:microchip
-LIBS:analog_switches
-LIBS:motorola
-LIBS:texas
-LIBS:intel
-LIBS:audio
-LIBS:interface
-LIBS:digital-audio
-LIBS:philips
-LIBS:display
-LIBS:cypress
-LIBS:siliconi
-LIBS:opto
-LIBS:atmel
-LIBS:contrib
-LIBS:valves
 LIBS:mirobot
 LIBS:Mirobot-cache
@@
 $EndComp
 $Comp
-L GND #PWR27
+L GND #PWR021
 U 1 1 56A07466
 P 3875 3550
-F 0 "#PWR27" H 3875 3300 60  0001 C CNN
+F 0 "#PWR021" H 3875 3300 60  0001 C CNN
 F 1 "GND" H 3875 3400 60  0000 C CNN
 F 2 "" H 3875 3550 60  0000 C CNN
@@
 $EndComp
 $Comp
-L VSS #PWR31
+L VSS #PWR022
 U 1 1 56A0746C
 P 5200 2925
-F 0 "#PWR31" H 5200 2775 60  0001 C CNN
+F 0 "#PWR022" H 5200 2775 60  0001 C CNN
 F 1 "VSS" H 5200 3075 60  0000 C CNN
 F 2 "" H 5200 2925 60  0000 C CNN
@@
 $EndComp
 $Comp
-L PWR_FLAG #FLG1
+L PWR_FLAG #FLG023
 U 1 1 56A07CE8
 P 3950 6375
-F 0 "#FLG1" H 3950 6470 30  0001 C CNN
+F 0 "#FLG023" H 3950 6470 30  0001 C CNN
 F 1 "PWR_FLAG" H 3950 6555 30  0000 C CNN
 F 2 "" H 3950 6375 60  0000 C CNN
@@
 $EndComp
 $Comp
-L PWR_FLAG #FLG2
+L PWR_FLAG #FLG024
 U 1 1 56A07CEE
 P 4350 6375
-F 0 "#FLG2" H 4350 6470 30  0001 C CNN
+F 0 "#FLG024" H 4350 6470 30  0001 C CNN
 F 1 "PWR_FLAG" H 4350 6555 30  0000 C CNN
 F 2 "" H 4350 6375 60  0000 C CNN
@@
 $EndComp
 $Comp
-L PWR_FLAG #FLG3
+L PWR_FLAG #FLG025
 U 1 1 56A07CF4
 P 4750 6375
-F 0 "#FLG3" H 4750 6470 30  0001 C CNN
+F 0 "#FLG025" H 4750 6470 30  0001 C CNN
 F 1 "PWR_FLAG" H 4750 6555 30  0000 C CNN
 F 2 "" H 4750 6375 60  0000 C CNN
@@
 $EndComp
 $Comp
-L GND #PWR30
+L GND #PWR026
 U 1 1 56A07CFA
 P 4750 6550
-F 0 "#PWR30" H 4750 6300 60  0001 C CNN
+F 0 "#PWR026" H 4750 6300 60  0001 C CNN
 F 1 "GND" H 4750 6400 60  0000 C CNN
 F 2 "" H 4750 6550 60  0000 C CNN
@@
 $EndComp
 $Comp
-L VSS #PWR29
+L VSS #PWR027
 U 1 1 56A07D00
 P 4350 6550
-F 0 "#PWR29" H 4350 6400 60  0001 C CNN
+F 0 "#PWR027" H 4350 6400 60  0001 C CNN
 F 1 "VSS" H 4350 6700 60  0000 C CNN
 F 2 "" H 4350 6550 60  0000 C CNN
@@
 $EndComp
 $Comp
-L +3V3 #PWR28
+L +3V3 #PWR028
 U 1 1 56A07D06
 P 3950 6550
-F 0 "#PWR28" H 3950 6400 60  0001 C CNN
+F 0 "#PWR028" H 3950 6400 60  0001 C CNN
 F 1 "+3V3" H 3950 6690 60  0000 C CNN
 F 2 "" H 3950 6550 60  0000 C CNN
@@
 $EndComp
 $Comp
-L GND #PWR22
-U 1 1 56A07D0C
-P 2275 6700
-F 0 "#PWR22" H 2275 6450 60  0001 C CNN
-F 1 "GND" H 2275 6550 60  0000 C CNN
-F 2 "" H 2275 6700 60  0000 C CNN
-F 3 "" H 2275 6700 60  0000 C CNN
-	1    2275 6700
-	1    0    0    -1
-$EndComp
-$Comp
-L GND #PWR24
-U 1 1 56A07D12
-P 2725 6700
-F 0 "#PWR24" H 2725 6450 60  0001 C CNN
-F 1 "GND" H 2725 6550 60  0000 C CNN
-F 2 "" H 2725 6700 60  0000 C CNN
-F 3 "" H 2725 6700 60  0000 C CNN
-	1    2725 6700
-	1    0    0    -1
-$EndComp
-$Comp
-L VSS #PWR21
-U 1 1 56A07D18
-P 2275 6025
-F 0 "#PWR21" H 2275 5875 60  0001 C CNN
-F 1 "VSS" H 2275 6175 60  0000 C CNN
-F 2 "" H 2275 6025 60  0000 C CNN
-F 3 "" H 2275 6025 60  0000 C CNN
-	1    2275 6025
-	1    0    0    -1
-$EndComp
-$Comp
-L +3V3 #PWR23
-U 1 1 56A07D1E
-P 2725 6025
-F 0 "#PWR23" H 2725 5875 60  0001 C CNN
-F 1 "+3V3" H 2725 6165 60  0000 C CNN
-F 2 "" H 2725 6025 60  0000 C CNN
-F 3 "" H 2725 6025 60  0000 C CNN
-	1    2725 6025
-	1    0    0    -1
-$EndComp
-$Comp
-L CP2 C4
-U 1 1 56A07D24
-P 2725 6350
-F 0 "C4" H 2775 6450 50  0000 L CNN
-F 1 "470uF" H 2775 6250 50  0000 L CNN
-F 2 "Capacitors_SMD:c_elec_8x10" H 2763 6200 30  0001 C CNN
-F 3 "" H 2725 6350 60  0000 C CNN
-	1    2725 6350
-	1    0    0    -1
-$EndComp
+L LD1117S33CTR U8
+U 1 1 56A07F5E
+P 6200 3225
+F 0 "U8" H 6200 3475 50  0000 C CNN
+F 1 "LD1117S33CTR" H 6200 3425 50  0000 C CNN
+F 2 "TO_SOT_Packages_SMD:SOT-223" H 6200 3325 50  0001 C CNN
+F 3 "" H 6200 3225 50  0000 C CNN
+	1    6200 3225
+	1    0    0    -1
+$EndComp
+$Comp
+L GND #PWR029
+U 1 1 56A083CE
+P 6200 3800
+F 0 "#PWR029" H 6200 3550 60  0001 C CNN
+F 1 "GND" H 6200 3650 60  0000 C CNN
+F 2 "" H 6200 3800 60  0000 C CNN
+F 3 "" H 6200 3800 60  0000 C CNN
+	1    6200 3800
+	1    0    0    -1
+$EndComp
+$Comp
+L +3V3 #PWR030
+U 1 1 56A0851B
+P 7400 2875
+F 0 "#PWR030" H 7400 2725 60  0001 C CNN
+F 1 "+3V3" H 7400 3015 60  0000 C CNN
+F 2 "" H 7400 2875 60  0000 C CNN
+F 3 "" H 7400 2875 60  0000 C CNN
+	1    7400 2875
+	1    0    0    -1
+$EndComp
+$Comp
+L C C6
+U 1 1 56A08564
+P 5575 3425
+F 0 "C6" H 5600 3525 50  0000 L CNN
+F 1 "10uF" H 5600 3325 50  0000 L CNN
+F 2 "Capacitors_SMD:C_0805" H 5613 3275 50  0001 C CNN
+F 3 "" H 5575 3425 50  0000 C CNN
+	1    5575 3425
+	1    0    0    -1
+$EndComp
+$Comp
+L C C7
+U 1 1 56A0859E
+P 6725 3425
+F 0 "C7" H 6750 3525 50  0000 L CNN
+F 1 "100uF" H 6750 3325 50  0000 L CNN
+F 2 "Capacitors_Tantalum_SMD:TantalC_SizeB_EIA-3528_Reflow" H 6763 3275 50  0001 C CNN
+F 3 "" H 6725 3425 50  0000 C CNN
+	1    6725 3425
+	1    0    0    -1
+$EndComp
+$Comp
+L C C8
+U 1 1 56A085E0
+P 7075 3425
+F 0 "C8" H 7100 3525 50  0000 L CNN
+F 1 "10uF" H 7100 3325 50  0000 L CNN
+F 2 "Capacitors_SMD:C_0805" H 7113 3275 50  0001 C CNN
+F 3 "" H 7075 3425 50  0000 C CNN
+	1    7075 3425
+	1    0    0    -1
+$EndComp
+Wire Wire Line
+	4925 3175 5800 3175
+Wire Wire Line
+	4125 3275 3675 3275
+Wire Wire Line
+	3675 3375 3875 3375
+Wire Wire Line
+	3875 3375 3875 3550
+Wire Wire Line
+	5200 3175 5200 2925
+Wire Wire Line
+	4750 6375 4750 6550
+Wire Wire Line
+	4350 6375 4350 6550
+Wire Wire Line
+	3950 6375 3950 6550
+Connection ~ 5200 3175
+Wire Wire Line
+	6200 3475 6200 3800
+Wire Wire Line
+	6600 3175 7400 3175
+Wire Wire Line
+	7400 3175 7400 2875
+Wire Wire Line
+	5575 3275 5575 3175
+Connection ~ 5575 3175
+Wire Wire Line
+	6725 3275 6725 3175
+Connection ~ 6725 3175
+Wire Wire Line
+	7075 3275 7075 3175
+Connection ~ 7075 3175
+Wire Wire Line
+	5575 3575 5575 3700
+Wire Wire Line
+	5575 3700 7075 3700
+Connection ~ 6200 3700
+Wire Wire Line
+	7075 3700 7075 3575
+Wire Wire Line
+	6725 3575 6725 3700
+Connection ~ 6725 3700
+Wire Wire Line
+	2275 6550 2275 6700
+Wire Wire Line
+	2275 6150 2275 6025
 $Comp
 L CP2 C3
@@
 $EndComp
 $Comp
-L GND #PWR26
-U 1 1 56A07D32
-P 3225 6700
-F 0 "#PWR26" H 3225 6450 60  0001 C CNN
-F 1 "GND" H 3225 6550 60  0000 C CNN
-F 2 "" H 3225 6700 60  0000 C CNN
-F 3 "" H 3225 6700 60  0000 C CNN
-	1    3225 6700
-	1    0    0    -1
-$EndComp
-$Comp
-L +3V3 #PWR25
-U 1 1 56A07D38
-P 3225 6025
-F 0 "#PWR25" H 3225 5875 60  0001 C CNN
-F 1 "+3V3" H 3225 6165 60  0000 C CNN
-F 2 "" H 3225 6025 60  0000 C CNN
-F 3 "" H 3225 6025 60  0000 C CNN
-	1    3225 6025
-	1    0    0    -1
-$EndComp
-$Comp
-L CP2 C5
-U 1 1 56A07D3E
-P 3225 6350
-F 0 "C5" H 3275 6450 50  0000 L CNN
-F 1 "100uF" H 3275 6250 50  0000 L CNN
-F 2 "Capacitors_Tantalum_SMD:TantalC_SizeB_EIA-3528_Reflow" H 3263 6200 30  0001 C CNN
-F 3 "" H 3225 6350 60  0000 C CNN
-	1    3225 6350
-	1    0    0    -1
-$EndComp
-$Comp
-L LD1117S33CTR U8
-U 1 1 56A07F5E
-P 6200 3225
-F 0 "U8" H 6200 3475 50  0000 C CNN
-F 1 "LD1117S33CTR" H 6200 3425 50  0000 C CNN
-F 2 "SOT-223" H 6200 3325 50  0000 C CNN
-F 3 "" H 6200 3225 50  0000 C CNN
-	1    6200 3225
-	1    0    0    -1
-$EndComp
-$Comp
-L GND #PWR32
-U 1 1 56A083CE
-P 6200 3800
-F 0 "#PWR32" H 6200 3550 60  0001 C CNN
-F 1 "GND" H 6200 3650 60  0000 C CNN
-F 2 "" H 6200 3800 60  0000 C CNN
-F 3 "" H 6200 3800 60  0000 C CNN
-	1    6200 3800
-	1    0    0    -1
-$EndComp
-$Comp
-L +3V3 #PWR33
-U 1 1 56A0851B
-P 7400 2875
-F 0 "#PWR33" H 7400 2725 60  0001 C CNN
-F 1 "+3V3" H 7400 3015 60  0000 C CNN
-F 2 "" H 7400 2875 60  0000 C CNN
-F 3 "" H 7400 2875 60  0000 C CNN
-	1    7400 2875
-	1    0    0    -1
-$EndComp
-$Comp
-L C C6
-U 1 1 56A08564
-P 5575 3425
-F 0 "C6" H 5600 3525 50  0000 L CNN
-F 1 "10uF" H 5600 3325 50  0000 L CNN
-F 2 "" H 5613 3275 50  0000 C CNN
-F 3 "" H 5575 3425 50  0000 C CNN
-	1    5575 3425
-	1    0    0    -1
-$EndComp
-$Comp
-L C C7
-U 1 1 56A0859E
-P 6725 3425
-F 0 "C7" H 6750 3525 50  0000 L CNN
-F 1 "100uF" H 6750 3325 50  0000 L CNN
-F 2 "" H 6763 3275 50  0000 C CNN
-F 3 "" H 6725 3425 50  0000 C CNN
-	1    6725 3425
-	1    0    0    -1
-$EndComp
-$Comp
-L C C8
-U 1 1 56A085E0
-P 7075 3425
-F 0 "C8" H 7100 3525 50  0000 L CNN
-F 1 "10uF" H 7100 3325 50  0000 L CNN
-F 2 "" H 7113 3275 50  0000 C CNN
-F 3 "" H 7075 3425 50  0000 C CNN
-	1    7075 3425
-	1    0    0    -1
-$EndComp
-Wire Wire Line
-	4925 3175 5800 3175
-Wire Wire Line
-	4125 3275 3675 3275
-Wire Wire Line
-	3675 3375 3875 3375
-Wire Wire Line
-	3875 3375 3875 3550
-Wire Wire Line
-	5200 3175 5200 2925
-Wire Wire Line
-	4750 6375 4750 6550
-Wire Wire Line
-	4350 6375 4350 6550
-Wire Wire Line
-	3950 6375 3950 6550
-Wire Wire Line
-	2275 6150 2275 6025
-Wire Wire Line
-	2275 6550 2275 6700
-Wire Wire Line
-	2725 6550 2725 6700
-Wire Wire Line
-	2725 6150 2725 6025
-Wire Wire Line
-	3225 6550 3225 6700
-Wire Wire Line
-	3225 6150 3225 6025
-Connection ~ 5200 3175
-Wire Wire Line
-	6200 3475 6200 3800
-Wire Wire Line
-	6600 3175 7400 3175
-Wire Wire Line
-	7400 3175 7400 2875
-Wire Wire Line
-	5575 3275 5575 3175
-Connection ~ 5575 3175
-Wire Wire Line
-	6725 3275 6725 3175
-Connection ~ 6725 3175
-Wire Wire Line
-	7075 3275 7075 3175
-Connection ~ 7075 3175
-Wire Wire Line
-	5575 3575 5575 3700
-Wire Wire Line
-	5575 3700 7075 3700
-Connection ~ 6200 3700
-Wire Wire Line
-	7075 3700 7075 3575
-Wire Wire Line
-	6725 3575 6725 3700
-Connection ~ 6725 3700
+L VSS #PWR031
+U 1 1 56A07D18
+P 2275 6025
+F 0 "#PWR031" H 2275 5875 60  0001 C CNN
+F 1 "VSS" H 2275 6175 60  0000 C CNN
+F 2 "" H 2275 6025 60  0000 C CNN
+F 3 "" H 2275 6025 60  0000 C CNN
+	1    2275 6025
+	1    0    0    -1
+$EndComp
+$Comp
+L GND #PWR032
+U 1 1 56A07D0C
+P 2275 6700
+F 0 "#PWR032" H 2275 6450 60  0001 C CNN
+F 1 "GND" H 2275 6550 60  0000 C CNN
+F 2 "" H 2275 6700 60  0000 C CNN
+F 3 "" H 2275 6700 60  0000 C CNN
+	1    2275 6700
+	1    0    0    -1
+$EndComp
 $EndSCHEMATC

Commit message: Update the BoM to embed it into KiCad
Parts:
- added F1: 1A, Fuse_Holders_and_Fuses:Fuse_SMD1206_Reflow, symbol FUSE
- BATT1: Description (none) -> JST XH 2 Pin Male Socket; Manfr. Part Number (MFP) (none) -> B2B-XH-A; Manufacturer Name (MFN) (none) -> JST; Required (none) -> y; Source1 (none) -> http://www.digikey.co.uk/product-detail/en/B2B-XH-A(LF)(SN)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
- C1: renamed from C3; footprint Capacitors_SMD:c_elec_8x10 -> Capacitors_SMD:c_elec_6.3x7.7; symbol CP2 -> CP1; Description (none) -> 470uF Electrolytic Capacitor SMD; Manufacturer Name (MFN) (none) -> Generic; Package ID (none) -> 6.3x7.7; Required (none) -> y
- C6, C8: Description (none) -> 10uF 0805 SMD Capacitor; Manufacturer Name (MFN) (none) -> Generic; Package ID (none) -> 0805; Required (none) -> y; Source2 (none) -> http://www.aliexpress.com/item/2012-0805-106K-10UF-25V-250p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
- C7: Description (none) -> 100uF Tantalum Capacitor; Manufacturer Name (MFN) (none) -> Generic; Package ID (none) -> 3528; Required (none) -> y
- SW3: footprint Mirobot:SMALL_SLIDE_SWITCH -> Custom:SMALL_SLIDE_SWITCH; Description (none) -> SPDT Slide Switch R/A; Manufacturer Name (MFN) (none) -> Generic; Required (none) -> y
- U8: Description (none) -> 3.3V Voltage Regulator; Manfr. Part Number (MFP) (none) -> LD1117S33CTR; Manufacturer Name (MFN) (none) -> ST; Package ID (none) -> SOT-223; Required (none) -> y; Source2 (none) -> http://www.aliexpress.com/item/high-quality-200PCS-AMS1117-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
Connections:
- net GND: now also SW3.4 (Shield)
- net VSS: now also F1.2; no longer SW3.1
- net at BATT1.2 (P2): now also SW3.1; no longer SW3.2
- net +5V: now reaches SW3.3
- new net: F1.1, SW3.2
Other:
- moved on the sheet: BATT1, SW3
Changed lines of the file:
@@
 LIBS:memory
 LIBS:xilinx
-LIBS:mirobot
+LIBS:custom-symbols
 LIBS:Mirobot-cache
 EELAYER 25 0
@@
 L CONN_01X02 BATT1
 U 1 1 56A0745F
-P 3475 3325
-F 0 "BATT1" H 3475 3475 50  0000 C CNN
-F 1 "BATT" V 3575 3325 50  0000 C CNN
-F 2 "Pin_Headers:Pin_Header_Straight_1x02" H 3475 3325 60  0001 C CNN
-F 3 "" H 3475 3325 60  0000 C CNN
-	1    3475 3325
+P 2775 3325
+F 0 "BATT1" H 2775 3475 50  0000 C CNN
+F 1 "BATT" V 2875 3325 50  0000 C CNN
+F 2 "Pin_Headers:Pin_Header_Straight_1x02" H 2775 3325 60  0001 C CNN
+F 3 "http://www.jst-mfg.com/product/pdf/eng/eXH.pdf" H 2775 3325 60  0001 C CNN
+F 4 "JST XH 2 Pin Male Socket" H 2775 3325 60  0001 C CNN "Description"
+F 5 "JST" H 2775 3325 60  0001 C CNN "Manufacturer Name (MFN)"
+F 6 "B2B-XH-A" H 2775 3325 60  0001 C CNN "Manfr. Part Number (MFP)"
+F 7 "http://www.digikey.co.uk/product-detail/en/B2B-XH-A(LF)(SN)/455-2247-ND/1651045" H 2775 3325 60  0001 C CNN "Source1"
+F 8 "y" H 2775 3325 60  0001 C CNN "Required"
+	1    2775 3325
 	-1   0    0    1
 $EndComp
 $Comp
-L GND #PWR021
+L GND #PWR029
 U 1 1 56A07466
-P 3875 3550
-F 0 "#PWR021" H 3875 3300 60  0001 C CNN
-F 1 "GND" H 3875 3400 60  0000 C CNN
-F 2 "" H 3875 3550 60  0000 C CNN
-F 3 "" H 3875 3550 60  0000 C CNN
-	1    3875 3550
-	1    0    0    -1
-$EndComp
-$Comp
-L VSS #PWR022
+P 3175 3550
+F 0 "#PWR029" H 3175 3300 60  0001 C CNN
+F 1 "GND" H 3175 3400 60  0000 C CNN
+F 2 "" H 3175 3550 60  0000 C CNN
+F 3 "" H 3175 3550 60  0000 C CNN
+	1    3175 3550
+	1    0    0    -1
+$EndComp
+$Comp
+L VSS #PWR030
 U 1 1 56A0746C
 P 5200 2925
-F 0 "#PWR022" H 5200 2775 60  0001 C CNN
+F 0 "#PWR030" H 5200 2775 60  0001 C CNN
 F 1 "VSS" H 5200 3075 60  0000 C CNN
 F 2 "" H 5200 2925 60  0000 C CNN
@@
 L SWITCH_SPDT SW3
 U 1 1 56A07472
-P 4525 3275
-F 0 "SW3" H 4525 3525 60  0000 C CNN
-F 1 "POWER_SWITCH" H 4565 3025 59  0000 C CNN
-F 2 "Mirobot:SMALL_SLIDE_SWITCH" H 4525 3275 60  0001 C CNN
-F 3 "" H 4525 3275 60  0000 C CNN
-	1    4525 3275
-	1    0    0    -1
-$EndComp
-$Comp
-L PWR_FLAG #FLG023
+P 3825 3175
+F 0 "SW3" H 4050 3425 60  0000 C CNN
+F 1 "POWER_SWITCH" H 3865 2925 59  0000 C CNN
+F 2 "Custom:SMALL_SLIDE_SWITCH" H 3825 3175 60  0001 C CNN
+F 3 "" H 3825 3175 60  0000 C CNN
+F 4 "SPDT Slide Switch R/A" H 3825 3175 60  0001 C CNN "Description"
+F 5 "Generic" H 3825 3175 60  0001 C CNN "Manufacturer Name (MFN)"
+F 6 "y" H 3825 3175 60  0001 C CNN "Required"
+	1    3825 3175
+	-1   0    0    1
+$EndComp
+$Comp
+L PWR_FLAG #FLG031
 U 1 1 56A07CE8
 P 3950 6375
-F 0 "#FLG023" H 3950 6470 30  0001 C CNN
+F 0 "#FLG031" H 3950 6470 30  0001 C CNN
 F 1 "PWR_FLAG" H 3950 6555 30  0000 C CNN
 F 2 "" H 3950 6375 60  0000 C CNN
@@
 $EndComp
 $Comp
-L PWR_FLAG #FLG024
+L PWR_FLAG #FLG032
 U 1 1 56A07CEE
 P 4350 6375
-F 0 "#FLG024" H 4350 6470 30  0001 C CNN
+F 0 "#FLG032" H 4350 6470 30  0001 C CNN
 F 1 "PWR_FLAG" H 4350 6555 30  0000 C CNN
 F 2 "" H 4350 6375 60  0000 C CNN
@@
 $EndComp
 $Comp
-L PWR_FLAG #FLG025
+L PWR_FLAG #FLG033
 U 1 1 56A07CF4
 P 4750 6375
-F 0 "#FLG025" H 4750 6470 30  0001 C CNN
+F 0 "#FLG033" H 4750 6470 30  0001 C CNN
 F 1 "PWR_FLAG" H 4750 6555 30  0000 C CNN
 F 2 "" H 4750 6375 60  0000 C CNN
@@
 $EndComp
 $Comp
-L GND #PWR026
+L GND #PWR034
 U 1 1 56A07CFA
 P 4750 6550
-F 0 "#PWR026" H 4750 6300 60  0001 C CNN
+F 0 "#PWR034" H 4750 6300 60  0001 C CNN
 F 1 "GND" H 4750 6400 60  0000 C CNN
 F 2 "" H 4750 6550 60  0000 C CNN
@@
 $EndComp
 $Comp
-L VSS #PWR027
+L VSS #PWR035
 U 1 1 56A07D00
 P 4350 6550
-F 0 "#PWR027" H 4350 6400 60  0001 C CNN
+F 0 "#PWR035" H 4350 6400 60  0001 C CNN
 F 1 "VSS" H 4350 6700 60  0000 C CNN
 F 2 "" H 4350 6550 60  0000 C CNN
@@
 $EndComp
 $Comp
-L +3V3 #PWR028
+L +3V3 #PWR036
 U 1 1 56A07D06
 P 3950 6550
-F 0 "#PWR028" H 3950 6400 60  0001 C CNN
+F 0 "#PWR036" H 3950 6400 60  0001 C CNN
 F 1 "+3V3" H 3950 6690 60  0000 C CNN
 F 2 "" H 3950 6550 60  0000 C CNN
@@
 F 1 "LD1117S33CTR" H 6200 3425 50  0000 C CNN
 F 2 "TO_SOT_Packages_SMD:SOT-223" H 6200 3325 50  0001 C CNN
-F 3 "" H 6200 3225 50  0000 C CNN
+F 3 "http://www.st.com/web/en/resource/technical/document/datasheet/CD00000544.pdf" H 6200 3225 50  0001 C CNN
+F 4 "3.3V Voltage Regulator" H 6200 3225 60  0001 C CNN "Description"
+F 5 "SOT-223" H 6200 3225 60  0001 C CNN "Package ID"
+F 6 "ST" H 6200 3225 60  0001 C CNN "Manufacturer Name (MFN)"
+F 7 "LD1117S33CTR" H 6200 3225 60  0001 C CNN "Manfr. Part Number (MFP)"
+F 8 "http://www.aliexpress.com/item/high-quality-200PCS-AMS1117-3-3V-AMS1117-1117-3-3V-1A-Regulator-LDO-SOT-223-Special/32603003633.html" H 6200 3225 60  0001 C CNN "Source2"
+F 9 "y" H 6200 3225 60  0001 C CNN "Required"
 	1    6200 3225
 	1    0    0    -1
 $EndComp
 $Comp
-L GND #PWR029
+L GND #PWR037
 U 1 1 56A083CE
 P 6200 3800
-F 0 "#PWR029" H 6200 3550 60  0001 C CNN
+F 0 "#PWR037" H 6200 3550 60  0001 C CNN
 F 1 "GND" H 6200 3650 60  0000 C CNN
 F 2 "" H 6200 3800 60  0000 C CNN
@@
 $EndComp
 $Comp
-L +3V3 #PWR030
+L +3V3 #PWR038
 U 1 1 56A0851B
 P 7400 2875
-F 0 "#PWR030" H 7400 2725 60  0001 C CNN
+F 0 "#PWR038" H 7400 2725 60  0001 C CNN
 F 1 "+3V3" H 7400 3015 60  0000 C CNN
 F 2 "" H 7400 2875 60  0000 C CNN
@@
 F 2 "Capacitors_SMD:C_0805" H 5613 3275 50  0001 C CNN
 F 3 "" H 5575 3425 50  0000 C CNN
+F 4 "10uF 0805 SMD Capacitor" H 5575 3425 60  0001 C CNN "Description"
+F 5 "0805" H 5575 3425 60  0001 C CNN "Package ID"
+F 6 "Generic" H 5575 3425 60  0001 C CNN "Manufacturer Name (MFN)"
+F 7 "http://www.aliexpress.com/item/2012-0805-106K-10UF-25V-250pcs-Original-authentic-and-new-Free-Shipping/32590605733.html" H 5575 3425 60  0001 C CNN "Source2"
+F 8 "y" H 5575 3425 60  0001 C CNN "Required"
 	1    5575 3425
 	1    0    0    -1
@@
 F 2 "Capacitors_Tantalum_SMD:TantalC_SizeB_EIA-3528_Reflow" H 6763 3275 50  0001 C CNN
 F 3 "" H 6725 3425 50  0000 C CNN
+F 4 "100uF Tantalum Capacitor" H 6725 3425 60  0001 C CNN "Description"
+F 5 "3528" H 6725 3425 60  0001 C CNN "Package ID"
+F 6 "Generic" H 6725 3425 60  0001 C CNN "Manufacturer Name (MFN)"
+F 7 "y" H 6725 3425 60  0001 C CNN "Required"
 	1    6725 3425
 	1    0    0    -1
@@
 F 2 "Capacitors_SMD:C_0805" H 7113 3275 50  0001 C CNN
 F 3 "" H 7075 3425 50  0000 C CNN
+F 4 "10uF 0805 SMD Capacitor" H 5575 3425 60  0001 C CNN "Description"
+F 5 "0805" H 5575 3425 60  0001 C CNN "Package ID"
+F 6 "Generic" H 5575 3425 60  0001 C CNN "Manufacturer Name (MFN)"
+F 7 "http://www.aliexpress.com/item/2012-0805-106K-10UF-25V-250pcs-Original-authentic-and-new-Free-Shipping/32590605733.html" H 7075 3425 60  0001 C CNN "Source2"
+F 8 "y" H 5575 3425 60  0001 C CNN "Required"
 	1    7075 3425
 	1    0    0    -1
@@
 	4925 3175 5800 3175
 Wire Wire Line
-	4125 3275 3675 3275
-Wire Wire Line
-	3675 3375 3875 3375
-Wire Wire Line
-	3875 3375 3875 3550
+	3425 3275 2975 3275
+Wire Wire Line
+	2975 3375 3175 3375
+Wire Wire Line
+	3175 3375 3175 3550
 Wire Wire Line
 	5200 3175 5200 2925
@@
 Connection ~ 6725 3700
 Wire Wire Line
-	2275 6550 2275 6700
-Wire Wire Line
-	2275 6150 2275 6025
-$Comp
-L CP2 C3
+	2275 6500 2275 6700
+Wire Wire Line
+	2275 6200 2275 6025
+$Comp
+L CP1 C1
 U 1 1 56A07D2B
 P 2275 6350
-F 0 "C3" H 2325 6450 50  0000 L CNN
+F 0 "C1" H 2325 6450 50  0000 L CNN
 F 1 "470uF" H 2325 6250 50  0000 L CNN
-F 2 "Capacitors_SMD:c_elec_8x10" H 2313 6200 30  0001 C CNN
+F 2 "Capacitors_SMD:c_elec_6.3x7.7" H 2313 6200 30  0001 C CNN
 F 3 "" H 2275 6350 60  0000 C CNN
+F 4 "470uF Electrolytic Capacitor SMD" H 2275 6350 60  0001 C CNN "Description"
+F 5 "6.3x7.7" H 2275 6350 60  0001 C CNN "Package ID"
+F 6 "Generic" H 2275 6350 60  0001 C CNN "Manufacturer Name (MFN)"
+F 7 "y" H 2275 6350 60  0001 C CNN "Required"
 	1    2275 6350
 	1    0    0    -1
 $EndComp
 $Comp
-L VSS #PWR031
+L VSS #PWR039
 U 1 1 56A07D18
 P 2275 6025
-F 0 "#PWR031" H 2275 5875 60  0001 C CNN
+F 0 "#PWR039" H 2275 5875 60  0001 C CNN
 F 1 "VSS" H 2275 6175 60  0000 C CNN
 F 2 "" H 2275 6025 60  0000 C CNN
@@
 $EndComp
 $Comp
-L GND #PWR032
+L GND #PWR040
 U 1 1 56A07D0C
 P 2275 6700
-F 0 "#PWR032" H 2275 6450 60  0001 C CNN
+F 0 "#PWR040" H 2275 6450 60  0001 C CNN
 F 1 "GND" H 2275 6550 60  0000 C CNN
 F 2 "" H 2275 6700 60  0000 C CNN
@@
 	1    0    0    -1
 $EndComp
+Wire Wire Line
+	3425 3075 3175 3075
+Wire Wire Line
+	3175 3075 3175 2850
+$Comp
+L +5V #PWR041
+U 1 1 56B2F9C1
+P 3175 2850
+F 0 "#PWR041" H 3175 2700 60  0001 C CNN
+F 1 "+5V" H 3175 2990 60  0000 C CNN
+F 2 "" H 3175 2850 60  0000 C CNN
+F 3 "" H 3175 2850 60  0000 C CNN
+	1    3175 2850
+	1    0    0    -1
+$EndComp
+$Comp
+L FUSE F1
+U 1 1 56B2FD56
+P 4675 3175
+F 0 "F1" H 4775 3225 50  0000 C CNN
+F 1 "1A" H 4575 3125 50  0000 C CNN
+F 2 "Fuse_Holders_and_Fuses:Fuse_SMD1206_Reflow" H 4675 3175 50  0001 C CNN
+F 3 "" H 4675 3175 50  0000 C CNN
+F 4 "1A Resettable fuse" H 4675 3175 60  0001 C CNN "Description"
+F 5 "1206" H 4675 3175 60  0001 C CNN "Package ID"
+F 6 "http://www.aliexpress.com/item/3000pcs-R429001WRM-429001-Fast-Acting-fuse-1206-1A-Marking-FH-ID387227/32600482167.html" H 4675 3175 60  0001 C CNN "Source2"
+F 7 "y" H 4675 3175 60  0001 C CNN "Required"
+	1    4675 3175
+	1    0    0    -1
+$EndComp
+Wire Wire Line
+	4425 3175 4225 3175
+$Comp
+L GND #PWR042
+U 1 1 56B3E3A0
+P 4300 3550
+F 0 "#PWR042" H 4300 3300 60  0001 C CNN
+F 1 "GND" H 4300 3400 60  0000 C CNN
+F 2 "" H 4300 3550 60  0000 C CNN
+F 3 "" H 4300 3550 60  0000 C CNN
+	1    4300 3550
+	1    0    0    -1
+$EndComp
+Wire Wire Line
+	4225 3375 4300 3375
+Wire Wire Line
+	4300 3375 4300 3550
 $EndSCHEMATC
