File: LineFollow/LineFollow.sch (KiCad schematic (older format))
At the start: 12 parts, among them P1 CONN_01X04, U1 LEFT_SENSE, U2 RIGHT_SENSE

Commit message: Updated for version 2.0f
Parts:
- removed LED1: LEFT_LED, Mirobot:SIDE-LED, symbol LED
- removed LED2: RIGHT_LED, Mirobot:SIDE-LED, symbol LED
- added LED1: LEFT_LED, Mirobot:SIDE-LED, symbol SIDE_LED
- added LED2: RIGHT_LED, Mirobot:SIDE-LED, symbol SIDE_LED
- R1, R3: value 220 -> 160
Connections:
- net GND: now also U1.2, U2.2, LED1.1, LED2.1; no longer U1.1, U2.1
- net at R1.1: now also LED1.2
- net at R3.1: now also LED2.2
- net at P1.3 (P3), R2.1: now also U1.1; no longer U1.2
- net at P1.4 (P4), R4.1: now also U2.1; no longer U2.2
Changed lines of the file:
@@
 $EndDescr
-$Comp
-L LED LED1
-U 1 1 55718A14
-P 5275 3575
-F 0 "LED1" H 5275 3675 50  0000 C CNN
-F 1 "LEFT_LED" H 5275 3475 50  0000 C CNN
-F 2 "Mirobot:SIDE-LED" H 5275 3575 60  0001 C CNN
-F 3 "" H 5275 3575 60  0000 C CNN
-	1    5275 3575
-	1    0    0    -1
-$EndComp
-$Comp
-L LED LED2
-U 1 1 55718A79
-P 7925 3575
-F 0 "LED2" H 7925 3675 50  0000 C CNN
-F 1 "RIGHT_LED" H 7925 3475 50  0000 C CNN
-F 2 "Mirobot:SIDE-LED" H 7925 3575 60  0001 C CNN
-F 3 "" H 7925 3575 60  0000 C CNN
-	1    7925 3575
-	1    0    0    -1
-$EndComp
 $Comp
 L R R1
@@
 P 4500 3575
 F 0 "R1" V 4580 3575 50  0000 C CNN
-F 1 "220" V 4507 3576 50  0000 C CNN
+F 1 "160" V 4507 3576 50  0000 C CNN
 F 2 "Resistors_SMD:R_0603" V 4430 3575 30  0001 C CNN
 F 3 "" H 4500 3575 30  0000 C CNN
@@
 P 7125 3575
 F 0 "R3" V 7205 3575 50  0000 C CNN
-F 1 "220" V 7132 3576 50  0000 C CNN
+F 1 "160" V 7132 3576 50  0000 C CNN
 F 2 "Resistors_SMD:R_0603" V 7055 3575 30  0001 C CNN
 F 3 "" H 7125 3575 30  0000 C CNN
@@
 F 3 "" H 5200 4300 60  0000 C CNN
 	1    5200 4300
-	1    0    0    -1
+	-1   0    0    -1
 $EndComp
 $Comp
@@
 F 3 "" H 7850 4300 60  0000 C CNN
 	1    7850 4300
-	1    0    0    -1
+	-1   0    0    -1
 $EndComp
 Wire Wire Line
@@
 	5875 4525 8275 4525
 Wire Wire Line
-	5475 3575 5875 3575
+	5350 3575 5875 3575
 Wire Wire Line
 	5875 3575 5875 4325
@@
 	7375 3575 7725 3575
 Wire Wire Line
-	8125 3575 8275 3575
+	8000 3575 8275 3575
 Connection ~ 8275 4300
 $Comp
@@
 	1    0    0    -1
 $EndComp
+$Comp
+L SIDE_LED LED2
+U 1 1 55B22939
+P 7875 3575
+F 0 "LED2" H 7875 3425 60  0000 C CNN
+F 1 "RIGHT_LED" H 7900 3775 60  0000 C CNN
+F 2 "Mirobot:SIDE-LED" H 7900 3575 60  0001 C CNN
+F 3 "" H 7900 3575 60  0000 C CNN
+	1    7875 3575
+	1    0    0    -1
+$EndComp
+$Comp
+L SIDE_LED LED1
+U 1 1 55B22A08
+P 5225 3575
+F 0 "LED1" H 5225 3425 60  0000 C CNN
+F 1 "LEFT_LED" H 5250 3775 60  0000 C CNN
+F 2 "Mirobot:SIDE-LED" H 5250 3575 60  0001 C CNN
+F 3 "" H 5250 3575 60  0000 C CNN
+	1    5225 3575
+	1    0    0    -1
+$EndComp

Commit message: Final production release for v2
Parts:
- U1, U2: footprint Mirobot:SIDE-LED -> Mirobot:SIDE-LED-REVERSED
Changed lines of the file:
@@
 F 0 "U1" H 5200 4200 60  0000 C CNN
 F 1 "LEFT_SENSE" H 5200 4600 60  0000 C CNN
-F 2 "Mirobot:SIDE-LED" H 5200 4300 60  0001 C CNN
+F 2 "Mirobot:SIDE-LED-REVERSED" H 5200 4300 60  0001 C CNN
 F 3 "" H 5200 4300 60  0000 C CNN
 	1    5200 4300
@@
 F 0 "U2" H 7850 4200 60  0000 C CNN
 F 1 "RIGHT_SENSE" H 7850 4600 60  0000 C CNN
-F 2 "Mirobot:SIDE-LED" H 7850 4300 60  0001 C CNN
+F 2 "Mirobot:SIDE-LED-REVERSED" H 7850 4300 60  0001 C CNN
 F 3 "" H 7850 4300 60  0000 C CNN
 	1    7850 4300
